Commit message: Reorganize

File: description/urdf/athena_arm.urdf.xacro (robot description, xacro)
@@ -10,21 +10,21 @@
   <!-- Macro Imports -->
   <!-- Import athena_arm macro -->
-  <xacro:include filename="$(find athena_arm_description)/urdf/athena_arm_description.urdf.xacro"/>
+  <xacro:include filename="$(find description)/urdf/description.urdf.xacro"/>
   <!-- Import mock ros2_control description -->
-  <xacro:include filename="$(find athena_arm_description)/ros2_control/mock.ros2_control.xacro" />
+  <xacro:include filename="$(find description)/ros2_control/mock.ros2_control.xacro" />
   <!-- Import smc ros2_control description -->
-  <xacro:include filename="$(find athena_arm_description)/ros2_control/smc.ros2_control.xacro" />
+  <xacro:include filename="$(find description)/ros2_control/smc.ros2_control.xacro" />
   <!-- Import talon ros2_control description -->
-  <xacro:include filename="$(find athena_arm_description)/ros2_control/talon.ros2_control.xacro" />
+  <xacro:include filename="$(find description)/ros2_control/talon.ros2_control.xacro" />
   <!-- Import rmd ros2_control description -->
-  <xacro:include filename="$(find athena_arm_description)/ros2_control/rmd.ros2_control.xacro" />
+  <xacro:include filename="$(find description)/ros2_control/rmd.ros2_control.xacro" />
   <!-- Import actuator ros2_control description -->
-  <xacro:include filename="$(find athena_arm_description)/ros2_control/actuator.ros2_control.xacro" />
+  <xacro:include filename="$(find description)/ros2_control/actuator.ros2_control.xacro" />
   <!-- Import odrive ros2_control description -->
-  <xacro:include filename="$(find athena_arm_description)/ros2_control/odrive.ros2_control.xacro" />
+  <xacro:include filename="$(find description)/ros2_control/odrive.ros2_control.xacro" />
   <!-- create link fixed to the "world" -->
   <link name="world"/>
   <!-- Contains description of arm -->
-  <xacro:athena_arm_description/>
+  <xacro:description/>
   <xacro:if value="$(arg use_mock_hardware)">     <!-- MOCK -->
     <xacro:mock_ros2_control name="mock"/>

File: description/urdf/athena_arm_description.urdf.xacro (robot description, xacro)
@@ -1,5 +1,5 @@
 <?xml version="1.0" encoding="utf-8"?>
 <robot xmlns:xacro="http://www.ros.org/wiki/xacro">
-  <xacro:macro name="athena_arm_description">
+  <xacro:macro name="description">
     <link
       name="base">
@@ -24,5 +24,5 @@
         <geometry>
           <mesh
-            filename="package://athena_arm_description/meshes/base.STL" />
+            filename="package://description/meshes/base.STL" />
         </geometry>
         <material
@@ -38,5 +38,5 @@
         <geometry>
           <mesh
-            filename="package://athena_arm_description/meshes/base.STL" />
+            filename="package://description/meshes/base.STL" />
         </geometry>
       </collision>
@@ -64,5 +64,5 @@
         <geometry>
           <mesh
-            filename="package://athena_arm_description/meshes/shoulder.STL" />
+            filename="package://description/meshes/shoulder.STL" />
         </geometry>
         <material
@@ -78,5 +78,5 @@
         <geometry>
           <mesh
-            filename="package://athena_arm_description/meshes/shoulder.STL" />
+            filename="package://description/meshes/shoulder.STL" />
         </geometry>
       </collision>
@@ -129,5 +129,5 @@
         <geometry>
           <mesh
-            filename="package://athena_arm_description/meshes/bicep.STL" />
+            filename="package://description/meshes/bicep.STL" />
         </geometry>
         <material
@@ -143,5 +143,5 @@
         <geometry>
           <mesh
-            filename="package://athena_arm_description/meshes/bicep.STL" />
+            filename="package://description/meshes/bicep.STL" />
         </geometry>
       </collision>
@@ -187,5 +187,5 @@
         <geometry>
           <mesh
-            filename="package://athena_arm_description/meshes/forearm.STL" />
+            filename="package://description/meshes/forearm.STL" />
         </geometry>
         <material
@@ -201,5 +201,5 @@
         <geometry>
           <mesh
-            filename="package://athena_arm_description/meshes/forearm.STL" />
+            filename="package://description/meshes/forearm.STL" />
         </geometry>
       </collision>
@@ -245,5 +245,5 @@
         <geometry>
           <mesh
-            filename="package://athena_arm_description/meshes/wrist_pitch.STL" />
+            filename="package://description/meshes/wrist_pitch.STL" />
         </geometry>
         <material
@@ -259,5 +259,5 @@
         <geometry>
           <mesh
-            filename="package://athena_arm_description/meshes/wrist_pitch.STL" />
+            filename="package://description/meshes/wrist_pitch.STL" />
         </geometry>
       </collision>
@@ -303,5 +303,5 @@
         <geometry>
           <mesh
-            filename="package://athena_arm_description/meshes/wrist_roll.STL" />
+            filename="package://description/meshes/wrist_roll.STL" />
         </geometry>
         <material
@@ -317,5 +317,5 @@
         <geometry>
           <mesh
-            filename="package://athena_arm_description/meshes/wrist_roll.STL" />
+            filename="package://description/meshes/wrist_roll.STL" />
         </geometry>
       </collision>
@@ -361,5 +361,5 @@
         <geometry>
           <mesh
-            filename="package://athena_arm_description/meshes/gripper_claw.STL" />
+            filename="package://description/meshes/gripper_claw.STL" />
         </geometry>
         <material
@@ -375,5 +375,5 @@
         <geometry>
           <mesh
-            filename="package://athena_arm_description/meshes/gripper_claw.STL" />
+            filename="package://description/meshes/gripper_claw.STL" />
         </geometry>
       </collision>
@@ -419,5 +419,5 @@
         <geometry>
           <mesh
-            filename="package://athena_arm_description/meshes/actuator.STL" />
+            filename="package://description/meshes/actuator.STL" />
         </geometry>
         <material
@@ -433,5 +433,5 @@
         <geometry>
           <mesh
-            filename="package://athena_arm_description/meshes/actuator.STL" />
+            filename="package://description/meshes/actuator.STL" />
         </geometry>
       </collision>

File: description/urdf/athena_drive.urdf.xacro (robot description, xacro)
@@ -8,6 +8,6 @@
   <xacro:arg name="sim_gazebo" default="true"/>
   <xacro:arg name="simulation_controllers" default=""/>
-  <xacro:include filename="$(find athena_drive_description)/urdf/athena_drive/athena_drive_macro.xacro"/>
-  <xacro:include filename="$(find athena_drive_description)/urdf/athena_drive/athena_drive_macro.ros2_control.xacro"/>
+  <xacro:include filename="$(find description)/urdf/athena_drive/athena_drive_macro.xacro"/>
+  <xacro:include filename="$(find description)/urdf/athena_drive/athena_drive_macro.ros2_control.xacro"/>
   <!-- Load robot's macro with parameters -->
   <!-- set prefix if multiple robots are used -->
@@ -18,12 +18,12 @@
   -->
   <!-- Import athena_drive macro -->
-  <xacro:include filename="$(find athena_drive_description)/urdf/athena_drive_description.urdf.xacro"/>
+  <xacro:include filename="$(find description)/urdf/description.urdf.xacro"/>
   <!-- Import rmd ros2_control description -->
-  <xacro:include filename="$(find athena_drive_description)/ros2_control/rmd.ros2_control.xacro" />
+  <xacro:include filename="$(find description)/ros2_control/rmd.ros2_control.xacro" />
   <!-- Import odrive ros2_control description -->
-  <xacro:include filename="$(find athena_drive_description)/ros2_control/odrive.ros2_control.xacro" />
+  <xacro:include filename="$(find description)/ros2_control/odrive.ros2_control.xacro" />
   <!-- create link fixed to the "world" -->
   <link name="world"/>
-  <xacro:athena_drive_description/>
+  <xacro:description/>
   <xacro:if value="$(arg use_mock_hardware)">
     <xacro:athena_drive_ros2_control

File: description/urdf/athena_drive/athena_drive_macro.xacro (robot description, xacro)
@@ -1,6 +1,6 @@
 <?xml version="1.0" encoding="UTF-8"?>
 <robot xmlns:xacro="http://wiki.ros.org/xacro">
-  <xacro:include filename="$(find athena_drive_description)/urdf/common/inertials.xacro"/>
-  <xacro:include filename="$(find athena_drive_description)/urdf/common/materials.xacro"/>
+  <xacro:include filename="$(find description)/urdf/common/inertials.xacro"/>
+  <xacro:include filename="$(find description)/urdf/common/materials.xacro"/>
   <xacro:macro name="athena_drive" params="prefix parent *origin">
     <!-- LINKS -->
@@ -14,5 +14,5 @@
         <geometry>
           <cylinder length="0.3" radius="0.3"/>
-          <!--           <mesh filename="package://athena_drive_description/meshes/athena_drive/visual/base_link.dae" /> -->
+          <!--           <mesh filename="package://description/meshes/athena_drive/visual/base_link.dae" /> -->
         </geometry>
         <material name="black"/>
@@ -22,5 +22,5 @@
         <geometry>
           <cylinder length="0.3" radius="0.3"/>
-          <!--           <mesh filename="package://athena_drive_description/meshes/athena_drive/collision/base_link.stl" /> -->
+          <!--           <mesh filename="package://description/meshes/athena_drive/collision/base_link.stl" /> -->
         </geometry>
       </collision>
@@ -35,5 +35,5 @@
         <geometry>
           <cylinder length="0.3" radius="0.15"/>
-          <!--           <mesh filename="package://athena_drive_description/meshes/athena_drive/visual/link1.dae" /> -->
+          <!--           <mesh filename="package://description/meshes/athena_drive/visual/link1.dae" /> -->
         </geometry>
         <material name="blue"/>
@@ -43,5 +43,5 @@
         <geometry>
           <cylinder length="0.3" radius="0.15"/>
-          <!--           <mesh filename="package://athena_drive_description/meshes/athena_drive/collision/link1.stl" /> -->
+          <!--           <mesh filename="package://description/meshes/athena_drive/collision/link1.stl" /> -->
         </geometry>
         <material name="green"/>
@@ -57,5 +57,5 @@
         <geometry>
           <cylinder length="0.3" radius="0.15"/>
-          <!--           <mesh filename="package://athena_drive_description/meshes/athena_drive/visual/link2.dae" /> -->
+          <!--           <mesh filename="package://description/meshes/athena_drive/visual/link2.dae" /> -->
         </geometry>
         <material name="grey"/>
@@ -65,5 +65,5 @@
         <geometry>
           <cylinder length="0.3" radius="0.15"/>
-          <!--           <mesh filename="package://athena_drive_description/meshes/athena_drive/collision/link2.stl"  /> -->
+          <!--           <mesh filename="package://description/meshes/athena_drive/collision/link2.stl"  /> -->
         </geometry>
       </collision>
@@ -78,5 +78,5 @@
         <geometry>
           <cylinder length="0.2" radius="0.1"/>
-          <!--           <mesh filename="package://athena_drive_description/meshes/athena_drive/visual/link3.dae" /> -->
+          <!--           <mesh filename="package://description/meshes/athena_drive/visual/link3.dae" /> -->
         </geometry>
         <material name="orange"/>
@@ -86,5 +86,5 @@
         <geometry>
           <cylinder length="0.2" radius="0.1"/>
-          <!--           <mesh filename="package://athena_drive_description/meshes/athena_drive/collision/link3.stl"  /> -->
+          <!--           <mesh filename="package://description/meshes/athena_drive/collision/link3.stl"  /> -->
         </geometry>
       </collision>
@@ -99,5 +99,5 @@
         <geometry>
           <cylinder length="0.1" radius="0.1"/>
-          <!--           <mesh filename="package://athena_drive_description/meshes/athena_drive/visual/link4.dae" /> -->
+          <!--           <mesh filename="package://description/meshes/athena_drive/visual/link4.dae" /> -->
         </geometry>
         <material name="brown"/>
@@ -107,5 +107,5 @@
         <geometry>
           <cylinder length="0.1" radius="0.1"/>
-          <!--           <mesh filename="package://athena_drive_description/meshes/athena_drive/collision/link4.stl"  /> -->
+          <!--           <mesh filename="package://description/meshes/athena_drive/collision/link4.stl"  /> -->
         </geometry>
       </collision>
@@ -120,5 +120,5 @@
         <geometry>
           <cylinder length="0.15" radius="0.1"/>
-          <!--           <mesh filename="package://athena_drive_description/meshes/athena_drive/visual/link5.dae" /> -->
+          <!--           <mesh filename="package://description/meshes/athena_drive/visual/link5.dae" /> -->
         </geometry>
         <material name="red"/>
@@ -128,5 +128,5 @@
         <geometry>
           <cylinder length="0.15" radius="0.1"/>
-          <!--           <mesh filename="package://athena_drive_description/meshes/athena_drive/collision/link5.stl" /> -->
+          <!--           <mesh filename="package://description/meshes/athena_drive/collision/link5.stl" /> -->
         </geometry>
       </collision>
@@ -141,5 +141,5 @@
         <geometry>
           <cylinder length="0.05" radius="0.075"/>
-          <!--           <mesh filename="package://athena_drive_description/meshes/athena_drive/visual/link6.dae" /> -->
+          <!--           <mesh filename="package://description/meshes/athena_drive/visual/link6.dae" /> -->
         </geometry>
         <material name="white"/>
@@ -149,5 +149,5 @@
         <geometry>
           <cylinder length="0.05" radius="0.075"/>
-          <!--           <mesh filename="package://athena_drive_description/meshes/athena_drive/collision/link6.stl" /> -->
+          <!--           <mesh filename="package://description/meshes/athena_drive/collision/link6.stl" /> -->
         </geometry>
       </collision>
