Commit message: Reorganize

File: description/urdf/athena_drive_description.urdf.xacro (robot description, xacro)
@@ -4,5 +4,5 @@
      For more information, please see http://wiki.ros.org/sw_urdf_exporter -->
 <robot xmlns:xacro="http://www.ros.org/wiki/xacro">
-  <xacro:macro name="athena_drive_description">
+  <xacro:macro name="description">
     <link
       name="chassis_base_link">
@@ -27,19 +27,19 @@
         <geometry>
           <mesh
-            filename="package://athena_drive_description/meshes/chassis_base_link.STL" />
-        </geometry>
-        <material
-          name="">
-          <color
-            rgba="0.792156862745098 0.819607843137255 0.933333333333333 1" />
-        </material>
-      </visual>
-      <collision>
-        <origin
-          xyz="0 0 0"
-          rpy="0 0 0" />
-        <geometry>
-          <mesh
-            filename="package://athena_drive_description/meshes/chassis_base_link.STL" />
+            filename="package://description/meshes/chassis_base_link.STL" />
+        </geometry>
+        <material
+          name="">
+          <color
+            rgba="0.792156862745098 0.819607843137255 0.933333333333333 1" />
+        </material>
+      </visual>
+      <collision>
+        <origin
+          xyz="0 0 0"
+          rpy="0 0 0" />
+        <geometry>
+          <mesh
+            filename="package://description/meshes/chassis_base_link.STL" />
         </geometry>
       </collision>
@@ -67,5 +67,5 @@
         <geometry>
           <mesh
-            filename="package://athena_drive_description/meshes/suspension_left_link.STL" />
+            filename="package://description/meshes/suspension_left_link.STL" />
         </geometry>
         <material
@@ -81,5 +81,5 @@
         <geometry>
           <mesh
-            filename="package://athena_drive_description/meshes/suspension_left_link.STL" />
+            filename="package://description/meshes/suspension_left_link.STL" />
         </geometry>
       </collision>
@@ -132,19 +132,19 @@
         <geometry>
           <mesh
-            filename="package://athena_drive_description/meshes/swerve_front_link.STL" />
-        </geometry>
-        <material
-          name="">
-          <color
-            rgba="0.792156862745098 0.819607843137255 0.933333333333333 1" />
-        </material>
-      </visual>
-      <collision>
-        <origin
-          xyz="0 0 0"
-          rpy="0 0 0" />
-        <geometry>
-          <mesh
-            filename="package://athena_drive_description/meshes/swerve_front_link.STL" />
+            filename="package://description/meshes/swerve_front_link.STL" />
+        </geometry>
+        <material
+          name="">
+          <color
+            rgba="0.792156862745098 0.819607843137255 0.933333333333333 1" />
+        </material>
+      </visual>
+      <collision>
+        <origin
+          xyz="0 0 0"
+          rpy="0 0 0" />
+        <geometry>
+          <mesh
+            filename="package://description/meshes/swerve_front_link.STL" />
         </geometry>
       </collision>
@@ -190,5 +190,5 @@
         <geometry>
           <mesh
-            filename="package://athena_drive_description/meshes/swerve_module_front_link.STL" />
+            filename="package://description/meshes/swerve_module_front_link.STL" />
         </geometry>
         <material
@@ -204,5 +204,5 @@
         <geometry>
           <mesh
-            filename="package://athena_drive_description/meshes/swerve_module_front_link.STL" />
+            filename="package://description/meshes/swerve_module_front_link.STL" />
         </geometry>
       </collision>
@@ -248,19 +248,19 @@
         <geometry>
           <mesh
-            filename="package://athena_drive_description/meshes/bracket_front_link.STL" />
-        </geometry>
-        <material
-          name="">
-          <color
-            rgba="0.792156862745098 0.819607843137255 0.933333333333333 1" />
-        </material>
-      </visual>
-      <collision>
-        <origin
-          xyz="0 0 0"
-          rpy="0 0 0" />
-        <geometry>
-          <mesh
-            filename="package://athena_drive_description/meshes/bracket_front_link.STL" />
+            filename="package://description/meshes/bracket_front_link.STL" />
+        </geometry>
+        <material
+          name="">
+          <color
+            rgba="0.792156862745098 0.819607843137255 0.933333333333333 1" />
+        </material>
+      </visual>
+      <collision>
+        <origin
+          xyz="0 0 0"
+          rpy="0 0 0" />
+        <geometry>
+          <mesh
+            filename="package://description/meshes/bracket_front_link.STL" />
         </geometry>
       </collision>
@@ -301,5 +301,5 @@
         <geometry>
           <mesh
-            filename="package://athena_drive_description/meshes/wheel_front_link.STL" />
+            filename="package://description/meshes/wheel_front_link.STL" />
         </geometry>
         <material
@@ -315,5 +315,5 @@
         <geometry>
           <mesh
-            filename="package://athena_drive_description/meshes/wheel_front_link.STL" />
+            filename="package://description/meshes/wheel_front_link.STL" />
         </geometry>
       </collision>
@@ -359,19 +359,19 @@
         <geometry>
           <mesh
-            filename="package://athena_drive_description/meshes/swerve_back_link.STL" />
-        </geometry>
-        <material
-          name="">
-          <color
-            rgba="0.792156862745098 0.819607843137255 0.933333333333333 1" />
-        </material>
-      </visual>
-      <collision>
-        <origin
-          xyz="0 0 0"
-          rpy="0 0 0" />
-        <geometry>
-          <mesh
-            filename="package://athena_drive_description/meshes/swerve_back_link.STL" />
+            filename="package://description/meshes/swerve_back_link.STL" />
+        </geometry>
+        <material
+          name="">
+          <color
+            rgba="0.792156862745098 0.819607843137255 0.933333333333333 1" />
+        </material>
+      </visual>
+      <collision>
+        <origin
+          xyz="0 0 0"
+          rpy="0 0 0" />
+        <geometry>
+          <mesh
+            filename="package://description/meshes/swerve_back_link.STL" />
         </geometry>
       </collision>
@@ -417,19 +417,19 @@
         <geometry>
           <mesh
-            filename="package://athena_drive_description/meshes/swerve_module_back_link.STL" />
-        </geometry>
-        <material
-          name="">
-          <color
-            rgba="0.792156862745098 0.819607843137255 0.933333333333333 1" />
-        </material>
-      </visual>
-      <collision>
-        <origin
-          xyz="0 0 0"
-          rpy="0 0 0" />
-        <geometry>
-          <mesh
-            filename="package://athena_drive_description/meshes/swerve_module_back_link.STL" />
+            filename="package://description/meshes/swerve_module_back_link.STL" />
+        </geometry>
+        <material
+          name="">
+          <color
+            rgba="0.792156862745098 0.819607843137255 0.933333333333333 1" />
+        </material>
+      </visual>
+      <collision>
+        <origin
+          xyz="0 0 0"
+          rpy="0 0 0" />
+        <geometry>
+          <mesh
+            filename="package://description/meshes/swerve_module_back_link.STL" />
         </geometry>
       </collision>
@@ -475,19 +475,19 @@
         <geometry>
           <mesh
-            filename="package://athena_drive_description/meshes/bracket_back_link.STL" />
-        </geometry>
-        <material
-          name="">
-          <color
-            rgba="0.792156862745098 0.819607843137255 0.933333333333333 1" />
-        </material>
-      </visual>
-      <collision>
-        <origin
-          xyz="0 0 0"
-          rpy="0 0 0" />
-        <geometry>
-          <mesh
-            filename="package://athena_drive_description/meshes/bracket_back_link.STL" />
+            filename="package://description/meshes/bracket_back_link.STL" />
+        </geometry>
+        <material
+          name="">
+          <color
+            rgba="0.792156862745098 0.819607843137255 0.933333333333333 1" />
+        </material>
+      </visual>
+      <collision>
+        <origin
+          xyz="0 0 0"
+          rpy="0 0 0" />
+        <geometry>
+          <mesh
+            filename="package://description/meshes/bracket_back_link.STL" />
         </geometry>
       </collision>
@@ -528,19 +528,19 @@
         <geometry>
           <mesh
-            filename="package://athena_drive_description/meshes/wheel_back_link.STL" />
-        </geometry>
-        <material
-          name="">
-          <color
-            rgba="0.792156862745098 0.819607843137255 0.933333333333333 1" />
-        </material>
-      </visual>
-      <collision>
-        <origin
-          xyz="0 0 0"
-          rpy="0 0 0" />
-        <geometry>
-          <mesh
-            filename="package://athena_drive_description/meshes/wheel_back_link.STL" />
+            filename="package://description/meshes/wheel_back_link.STL" />
+        </geometry>
+        <material
+          name="">
+          <color
+            rgba="0.792156862745098 0.819607843137255 0.933333333333333 1" />
+        </material>
+      </visual>
+      <collision>
+        <origin
+          xyz="0 0 0"
+          rpy="0 0 0" />
+        <geometry>
+          <mesh
+            filename="package://description/meshes/wheel_back_link.STL" />
         </geometry>
       </collision>
@@ -586,19 +586,19 @@
         <geometry>
           <mesh
-            filename="package://athena_drive_description/meshes/suspension_right_link.STL" />
-        </geometry>
-        <material
-          name="">
-          <color
-            rgba="0.792156862745098 0.819607843137255 0.933333333333333 1" />
-        </material>
-      </visual>
-      <collision>
-        <origin
-          xyz="0 0 0"
-          rpy="0 0 0" />
-        <geometry>
-          <mesh
-            filename="package://athena_drive_description/meshes/suspension_right_link.STL" />
+            filename="package://description/meshes/suspension_right_link.STL" />
+        </geometry>
+        <material
+          name="">
+          <color
+            rgba="0.792156862745098 0.819607843137255 0.933333333333333 1" />
+        </material>
+      </visual>
+      <collision>
+        <origin
+          xyz="0 0 0"
+          rpy="0 0 0" />
+        <geometry>
+          <mesh
+            filename="package://description/meshes/suspension_right_link.STL" />
         </geometry>
       </collision>
@@ -644,19 +644,19 @@
         <geometry>
           <mesh
-            filename="package://athena_drive_description/meshes/swerve_front2_link.STL" />
-        </geometry>
-        <material
-          name="">
-          <color
-            rgba="0.792156862745098 0.819607843137255 0.933333333333333 1" />
-        </material>
-      </visual>
-      <collision>
-        <origin
-          xyz="0 0 0"
-          rpy="0 0 0" />
-        <geometry>
-          <mesh
-            filename="package://athena_drive_description/meshes/swerve_front2_link.STL" />
+            filename="package://description/meshes/swerve_front2_link.STL" />
+        </geometry>
+        <material
+          name="">
+          <color
+            rgba="0.792156862745098 0.819607843137255 0.933333333333333 1" />
+        </material>
+      </visual>
+      <collision>
+        <origin
+          xyz="0 0 0"
+          rpy="0 0 0" />
+        <geometry>
+          <mesh
+            filename="package://description/meshes/swerve_front2_link.STL" />
         </geometry>
       </collision>
@@ -702,19 +702,19 @@
         <geometry>
           <mesh
-            filename="package://athena_drive_description/meshes/swerve_module_front2_link.STL" />
-        </geometry>
-        <material
-          name="">
-          <color
-            rgba="0.792156862745098 0.819607843137255 0.933333333333333 1" />
-        </material>
-      </visual>
-      <collision>
-        <origin
-          xyz="0 0 0"
-          rpy="0 0 0" />
-        <geometry>
-          <mesh
-            filename="package://athena_drive_description/meshes/swerve_module_front2_link.STL" />
+            filename="package://description/meshes/swerve_module_front2_link.STL" />
+        </geometry>
+        <material
+          name="">
+          <color
+            rgba="0.792156862745098 0.819607843137255 0.933333333333333 1" />
+        </material>
+      </visual>
+      <collision>
+        <origin
+          xyz="0 0 0"
+          rpy="0 0 0" />
+        <geometry>
+          <mesh
+            filename="package://description/meshes/swerve_module_front2_link.STL" />
         </geometry>
       </collision>
@@ -760,19 +760,19 @@
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