Commit message: changed suspension joints from revolute to fixed

File: src/description/urdf/athena_drive_description.urdf.xacro (robot description, xacro)
@@ -49,5 +49,5 @@
             </collision>
         </link>
-        <joint name="suspension_front_left_joint" type="revolute">
+        <joint name="suspension_front_left_joint" type="fixed">
             <origin xyz="0.61263 0.22146 -0.74592" rpy="1.5708 0 0.094743" />
             <parent link="chassis_base_link" />
@@ -304,5 +304,5 @@
             </collision>
         </link>
-        <joint name="suspension_front_right_joint" type="revolute">
+        <joint name="suspension_front_right_joint" type="fixed">
             <origin xyz="0.66803 -0.36146 -0.74592" rpy="1.5708 0 0.094743" />
             <parent link="chassis_base_link" />

Commit message: Consolidated and fixed URDF into single file, fixed issues related to axis to enable proper drive control (#1)
* Fixed simulation bugs to enable rover control in gazebo

* changed suspension joints from revolute to fixed

File: src/description/urdf/athena_drive_description.urdf.xacro (robot description, xacro)
@@ -4,1076 +4,537 @@
      For more information, please see http://wiki.ros.org/sw_urdf_exporter -->
 <robot xmlns:xacro="http://www.ros.org/wiki/xacro">
-  <xacro:macro name="description">
-    <link
-      name="chassis_base_link">
-      <inertial>
-        <origin
-          xyz="0.775305042176281 -0.0692748019047986 -0.475175318827691"
-          rpy="0 0 0" />
-        <mass
-          value="44.0454429414672" />
-        <inertia
-          ixx="1.41725466889743"
-          ixy="0.00803894609354262"
-          ixz="-1.19304822311593E-17"
-          iyy="1.33698338807128"
-          iyz="1.62926079635059E-16"
-          izz="2.58380655400253" />
-      </inertial>
-      <visual>
-        <origin
-          xyz="0 0 0"
-          rpy="0 0 0" />
-        <geometry>
-          <mesh
-            filename="package://description/meshes/chassis_base_link.STL" />
-        </geometry>
-        <material
-          name="">
-          <color
-            rgba="0.792156862745098 0.819607843137255 0.933333333333333 1" />
-        </material>
-      </visual>
-      <collision>
-        <origin
-          xyz="0 0 0"
-          rpy="0 0 0" />
-        <geometry>
-          <mesh
-            filename="package://description/meshes/chassis_base_link.STL" />
-        </geometry>
-      </collision>
-    </link>
-    <link
-      name="suspension_left_link">
-      <inertial>
-        <origin
-          xyz="0.099658 0.17786 0.012079"
-          rpy="0 0 0" />
-        <mass
-          value="0.81514" />
-        <inertia
-          ixx="0.0036237"
-          ixy="2.1053E-06"
-          ixz="-1.8807E-07"
-          iyy="0.034331"
-          iyz="-6.6719E-08"
-          izz="0.037876" />
-      </inertial>
-      <visual>
-        <origin
-          xyz="0 0 0"
-          rpy="0 0 0" />
-        <geometry>
-          <mesh
-            filename="package://description/meshes/suspension_left_link.STL" />
-        </geometry>
-        <material
-          name="">
-          <color
-            rgba="0.79216 0.81961 0.93333 1" />
-        </material>
-      </visual>
-      <collision>
-        <origin
-          xyz="0 0 0"
-          rpy="0 0 0" />
-        <geometry>
-          <mesh
-            filename="package://description/meshes/suspension_left_link.STL" />
-        </geometry>
-      </collision>
-    </link>
-    <!-- base_joint fixes base_link to the environment -->
-    <joint name="base_joint" type="fixed">
-      <parent link="world"/>
-      <child link="chassis_base_link"/>
-      <origin xyz="0 0 0" rpy="0 0 0"/>
-      <axis xyz="0 0 1"/>
-    </joint>
-    <joint
-      name="suspension_left_joint"
-      type="revolute">
-      <origin
-        xyz="0.61263 0.22146 -0.74592"
-        rpy="1.5708 0 0.094743" />
-      <parent
-        link="chassis_base_link" />
-      <child
-        link="suspension_left_link" />
-      <axis
-        xyz="0 0 -1" />
-      <limit
-        lower="-1.0471975512"
-        upper="1.0471975512"
-        effort="200"
-        velocity="3" />
-    </joint>
-    <link
-      name="swerve_front_link">
-      <inertial>
-        <origin
-          xyz="-0.0150723908729249 -0.0104708416933169 0.0599977306724315"
-          rpy="0 0 0" />
-        <mass
-          value="0.0539897173870708" />
-        <inertia
-          ixx="0.000103437060477465"
-          ixy="1.625957825095E-05"
-          ixz="1.84667466664483E-09"
-          iyy="0.00015935267908897"
-          iyz="-9.66551053737858E-10"
-          izz="8.16571493320534E-05" />
-      </inertial>
-      <visual>
-        <origin
-          xyz="0 0 0"
-          rpy="0 0 0" />
-        <geometry>
-          <mesh
-            filename="package://description/meshes/swerve_front_link.STL" />
-        </geometry>
-        <material
-          name="">
-          <color
-            rgba="0.792156862745098 0.819607843137255 0.933333333333333 1" />
-        </material>
-      </visual>
-      <collision>
-        <origin
-          xyz="0 0 0"
-          rpy="0 0 0" />
-        <geometry>
-          <mesh
-            filename="package://description/meshes/swerve_front_link.STL" />
-        </geometry>
-      </collision>
-    </link>
-    <joint
-      name="swerve_front_joint"
-      type="fixed">
-      <origin
-        xyz="-0.30502 0.067874 0.068599"
-        rpy="3.1416 0 3.1416" />
-      <parent
-        link="suspension_left_link" />
-      <child
-        link="swerve_front_link" />
-      <axis
-        xyz="0 0 0" />
-      <limit
-        lower="0"
-        upper="6.2832"
-        effort="200"
-        velocity="200" />
-    </joint>
-    <link
-      name="swerve_module_front_link">
-      <inertial>
-        <origin
-          xyz="-1.4988E-15 0.041875 2.2204E-16"
-          rpy="0 0 0" />
-        <mass
-          value="0.59412" />
-        <inertia
-          ixx="0.001058"
-          ixy="-3.6415E-36"
-          ixz="-4.3601E-37"
-          iyy="0.000433"
-          iyz="-2.3553E-22"
-          izz="0.001058" />
-      </inertial>
-      <visual>
-        <origin
-          xyz="0 0 0"
-          rpy="0 0 0" />
-        <geometry>
-          <mesh
-            filename="package://description/meshes/swerve_module_front_link.STL" />
-        </geometry>
-        <material
-          name="">
-          <color
-            rgba="0.79216 0.81961 0.93333 1" />
-        </material>
-      </visual>
-      <collision>
-        <origin
-          xyz="0 0 0"
-          rpy="0 0 0" />
-        <geometry>
-          <mesh
-            filename="package://description/meshes/swerve_module_front_link.STL" />
-        </geometry>
-      </collision>
-    </link>
-    <joint
-      name="swerve_module_front_left_joint"
-      type="revolute">
-      <origin
-        xyz="0 0 0.059903"
-        rpy="3.1416 0.094743 3.1416" />
-      <parent
-        link="swerve_front_link" />
-      <child
-        link="swerve_module_front_link" />
-      <axis
-        xyz="0 1 0" />
-      <limit
-        lower="0"
-        upper="6.2832"
-        effort="200"
-        velocity="3" />
-    </joint>
-    <link
-      name="bracket_front_link">
-      <inertial>
-        <origin
-          xyz="1.66533453693773E-16 0.0313698536921512 -0.0102283967385405"
-          rpy="0 0 0" />
-        <mass
-          value="0.064710634958827" />
-        <inertia
-          ixx="0.00034507967071994"
-          ixy="-6.70003061278152E-19"
-          ixz="2.50721752387273E-19"
-          iyy="6.46019700513441E-05"
-          iyz="5.56350874006337E-05"
-          izz="0.000344914371141864" />
-      </inertial>
-      <visual>
-        <origin
-          xyz="0 0 0"
-          rpy="0 0 0" />
-        <geometry>
-          <mesh
-            filename="package://description/meshes/bracket_front_link.STL" />
-        </geometry>
-        <material
-          name="">
-          <color
-            rgba="0.792156862745098 0.819607843137255 0.933333333333333 1" />
-        </material>
-      </visual>
-      <collision>
-        <origin
-          xyz="0 0 0"
-          rpy="0 0 0" />
-        <geometry>
-          <mesh
-            filename="package://description/meshes/bracket_front_link.STL" />
-        </geometry>
-      </collision>
-    </link>
-    <joint
-      name="bracket_front_joint"
-      type="fixed">
-      <origin
-        xyz="0.011719658421911 -0.128534743589743 -0.0584684115770519"
-        rpy="3.14159265358979 -0.0947430505373148 3.14159265358979" />
-      <parent
-        link="swerve_module_front_link" />
-      <child
-        link="bracket_front_link" />
-      <axis
-        xyz="0 0 0" />
-    </joint>
-    <link
-      name="wheel_front_link">
-      <inertial>
-        <origin
-          xyz="1.1102E-16 1.1102E-16 0.052423"
-          rpy="0 0 0" />
-        <mass
-          value="5.2824" />
-        <inertia
-          ixx="0.026006"
-          ixy="-2.6722E-33"
-          ixz="2.4503E-17"
-          iyy="0.026006"
-          iyz="-2.0265E-18"
-          izz="0.042334" />
-      </inertial>
-      <visual>
-        <origin
-          xyz="0 0 0"
-          rpy="0 0 0" />
-        <geometry>
-          <mesh
-            filename="package://description/meshes/wheel_front_link.STL" />
-        </geometry>
-        <material
-          name="">
-          <color
-            rgba="0.79216 0.81961 0.93333 1" />
-        </material>
-      </visual>
-      <collision>
-        <origin
-          xyz="0 0 0"
-          rpy="0 0 0" />
-        <geometry>
-          <mesh
-            filename="package://description/meshes/wheel_front_link.STL" />
-        </geometry>
-      </collision>
-    </link>
-    <joint
-      name="wheel_front_right_joint"
-      type="revolute">
-      <origin
-        xyz="0 -0.054545 -0.10628"
-        rpy="0 0 0" />
-      <parent
-        link="bracket_front_link" />
-      <child
-        link="wheel_front_link" />
-      <axis
-        xyz="0 0 -1" />
-      <limit
-        lower="0"
-        upper="6.2832"
-        effort="200"
-        velocity="3" />
-    </joint>
-    <link
-      name="swerve_back_link">
-      <inertial>
-        <origin
-          xyz="-0.0150723908729247 -0.0104708416933168 0.0599977306724315"
-          rpy="0 0 0" />
-        <mass
-          value="0.0539897173870708" />
-        <inertia
-          ixx="0.000103437060477465"
-          ixy="1.62595782509495E-05"
-          ixz="1.84667466674139E-09"
-          iyy="0.00015935267908897"
-          iyz="-9.66551053681107E-10"
-          izz="8.16571493320531E-05" />
-      </inertial>
-      <visual>
-        <origin
-          xyz="0 0 0"
-          rpy="0 0 0" />
-        <geometry>
-          <mesh
-            filename="package://description/meshes/swerve_back_link.STL" />
-        </geometry>
-        <material
-          name="">
-          <color
-            rgba="0.792156862745098 0.819607843137255 0.933333333333333 1" />
-        </material>
-      </visual>
-      <collision>
-        <origin
-          xyz="0 0 0"
-          rpy="0 0 0" />
-        <geometry>
-          <mesh
-            filename="package://description/meshes/swerve_back_link.STL" />
-        </geometry>
-      </collision>
-    </link>
-    <joint
-      name="swerve_back_joint"
-      type="fixed">
-      <origin
-        xyz="0.504296500310465 0.0678739512598524 -0.0501174912181417"
-        rpy="0 0 0" />
-      <parent
-        link="suspension_left_link" />
-      <child
-        link="swerve_back_link" />
-      <axis
-        xyz="0 0 0" />
-      <limit
-        lower="0"
-        upper="6.2832"
-        effort="200"
-        velocity="3" />
-    </joint>
-    <link
-      name="swerve_module_back_link">
-      <inertial>
-        <origin
-          xyz="-1.77635683940025E-15 0.041284522440529 5.55111512312578E-17"
-          rpy="0 0 0" />
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
Commit message: SDF creation and joystick integration with sim

File: src/description/urdf/athena_drive_description.urdf.xacro (robot description, xacro)
@@ -111,5 +111,5 @@
             <child link="steer_1_link" />
             <axis xyz="0 1 0" />
-            <limit lower="0" upper="6.2832" effort="200" velocity="3" />
+            <limit lower="-3.1416" upper="3.1416" effort="200" velocity="3" />
         </joint>
         <link name="wheel_bracket_1_link">
@@ -224,5 +224,5 @@
             <child link="steer_4_link" />
             <axis xyz="0 1 0" />
-            <limit lower="0" upper="6.2832" effort="200" velocity="3" />
+            <limit lower="-3.1416" upper="3.1416" effort="200" velocity="3" />
         </joint>
         <link name="wheel_bracket_4_link">
@@ -366,5 +366,5 @@
             <child link="steer_2_link" />
             <axis xyz="0 1 0" />
-            <limit lower="0" upper="6.2832" effort="200" velocity="3" />
+            <limit lower="-3.1416" upper="3.1416" effort="200" velocity="3" />
         </joint>
         <link name="wheel_bracket_2_link">
@@ -479,5 +479,5 @@
             <child link="steer_3_link" />
             <axis xyz="0 1 0" />
-            <limit lower="0" upper="6.28318530718" effort="200" velocity="3" />
+            <limit lower="-3.1416" upper="3.1416" effort="200" velocity="3" />
         </joint>
         <link name="wheel_bracket_3_link">
