Commit message: fix suspension naming

File: src/description/urdf/athena_drive/athena_drive_macro.ros2_control.xacro (robot description, xacro)
@@ -14,5 +14,5 @@
                 </xacro:unless>
             </hardware>
-            <joint name="${prefix}suspension_left_joint">
+            <joint name="${prefix}suspension_front_left_joint">
                 <command_interface name="position">
                     <param name="min">-1.0471975512</param>
@@ -24,5 +24,5 @@
                 <state_interface name="velocity"/>
             </joint>
-            <joint name="${prefix}suspension_right_joint">
+            <joint name="${prefix}suspension_front_right_joint">
                 <command_interface name="position">
                     <param name="min">-1.0471975512</param>

File: src/description/urdf/athena_drive/athena_drive_macro.xacro (robot description, xacro)
@@ -173,5 +173,5 @@
     </joint>
     <!-- joint 1 -->
-    <joint name="${prefix}suspension_left_joint" type="revolute">
+    <joint name="${prefix}suspension_front_left_joint" type="revolute">
       <origin xyz="0 0 0.3" rpy="${pi} 0 0"/>
       <parent link="${prefix}base_link"/>
@@ -213,5 +213,5 @@
     </joint>
     <!-- joint 6 -->
-    <joint name="${prefix}suspension_right_joint" type="revolute">
+    <joint name="${prefix}suspension_front_right_joint" type="revolute">
       <origin xyz="0.125 0 0" rpy="0 ${-pi/2} 0"/>
       <parent link="${prefix}link5"/>
@@ -221,5 +221,5 @@
     </joint>
     <!-- tool frame - fixed frame -->
-    <joint name="${prefix}suspension_right_joint-tool0" type="fixed">
+    <joint name="${prefix}suspension_front_right_joint-tool0" type="fixed">
       <parent link="${prefix}link6"/>
       <child link="${prefix}tool0"/>
