Commit message: refactor: Laser/Killswitch to CAN, move LED/Killswitch to drive
Address team lead feedback: Laser and Killswitch now use CAN protocol instead of GPIO. LED stays GPIO. All use gpio tags and gpio_command_controller. LED and Killswitch moved from science to drive subsystem. Added simulation fallback for development.

File: src/description/ros2_control/science/science.laser.ros2_control.xacro (robot description, xacro)
@@ -1,19 +1,18 @@
 <?xml version="1.0"?>
 <robot xmlns:xacro="http://www.ros.org/wiki/xacro">
-    <xacro:macro name="laser_ros2_control" params="name gpio_pin min_power:=0.0 max_power:=1.0">
+    <xacro:macro name="laser_ros2_control" params="name can_interface:=can0 can_id:=304">
+        <!-- CAN ID 0x130 = 304 decimal -->
         <ros2_control name="${name}" type="system">
             <hardware>
                 <plugin>laser_ros2_control/LaserHardwareInterface</plugin>
-                <param name="gpio_pin">${gpio_pin}</param>
-                <param name="min_power">${min_power}</param>
-                <param name="max_power">${max_power}</param>
+                <param name="can_interface">${can_interface}</param>
+                <param name="can_id">${can_id}</param>
             </hardware>
-            <joint name="${name}">
+            <gpio name="${name}">
                 <state_interface name="laser_state"/>
-                <state_interface name="power_level"/>
-                <state_interface name="is_ready"/>
+                <state_interface name="temperature"/>
+                <state_interface name="is_connected"/>
                 <command_interface name="laser_command"/>
-                <command_interface name="power_command"/>
-            </joint>
+            </gpio>
         </ros2_control>
     </xacro:macro>

File: src/description/urdf/athena_science.urdf.xacro (robot description, xacro)
@@ -8,6 +8,4 @@
   <xacro:include filename="$(find description)/ros2_control/science/science.talon.ros2_control.xacro"/>
   <xacro:include filename="$(find description)/ros2_control/science/science.laser.ros2_control.xacro"/>
-  <xacro:include filename="$(find description)/ros2_control/science/science.killswitch.ros2_control.xacro"/>
-  <xacro:include filename="$(find description)/ros2_control/science/science.led.ros2_control.xacro"/>
   <!-- create link fixed to the "world" -->
   <link name="world"/>
@@ -25,15 +23,6 @@
     <!-- Import talon ros2_control description -->
     <xacro:talon_ros2_control name="talon"/>
-    <!-- Import laser ros2_control description -->
-    <xacro:laser_ros2_control name="spectrometry_laser" gpio_pin="17"/>
-    <!-- Import killswitch ros2_control description -->
-    <xacro:killswitch_ros2_control
-      name="drive_killswitch"
-      button_gpio_pin="27"
-      main_power_gpio_pin="22"
-      jetson_power_gpio_pin="23"
-      all_power_gpio_pin="24"/>
-    <!-- Import LED ros2_control description -->
-    <xacro:led_ros2_control name="status_led" gpio_pin="25"/>
+    <!-- Import laser ros2_control description (CAN-based) -->
+    <xacro:laser_ros2_control name="spectrometry_laser"/>
   </xacro:unless>
 </robot>
