Commit message: heavy modifications to controller, working manual science controller implementation

File: src/description/ros2_control/science/science.servo.ros2_control.xacro (robot description, xacro)
@@ -7,9 +7,9 @@
                 <param name="update_rate">10</param> <!-- Hz -->
                 <param name="logger_rate">5</param> <!-- Hz -->
-                <param name="logger_state">1</param> <!-- 0 for off, 1 for on -->
+                <param name="logger_state">0</param> <!-- 0 for off, 1 for on -->
                 <param name="can_interface">can0</param>
                 <param name="can_id">0x80</param>
             </hardware>
-            <joint name="rack_and_pinion_left">
+            <joint name="servo_rack_and_pinion_l">
                 <param name="node_id">0x2</param>
                 <param name="gear_ratio">1</param>
@@ -17,5 +17,5 @@
                 <param name ="meters_per_deg">0.00016666666</param> <!-- (TODO) convert motor position in degrees to displacement in meters -->
                 <param name="servo_type">standard</param> <!-- standard or continuous -->
-                <param name="joint_type">prismatic</param> <!-- revolute or prismatic -->
+                <param name="joint_type">revolute</param> <!-- revolute or prismatic -->
                 <command_interface name="position"/>
                 <command_interface name="velocity"/>
@@ -23,5 +23,5 @@
                 <state_interface name="velocity"/>
             </joint>
-            <joint name="rack_and_pinion_right">
+            <joint name="servo_rack_and_pinion_r">
                 <param name="node_id">0x1</param>
                 <param name="gear_ratio">1</param>
@@ -29,5 +29,5 @@
                 <param name ="meters_per_deg">0.00016666666</param> <!-- (TODO) convert motor position in degrees to displacement in meters -->
                 <param name="servo_type">standard</param> <!-- standard or continuous -->
-                <param name="joint_type">prismatic</param> <!-- revolute or prismatic -->
+                <param name="joint_type">revolute</param> <!-- revolute or prismatic -->
                 <command_interface name="position"/>
                 <command_interface name="velocity"/>
@@ -35,6 +35,6 @@
                 <state_interface name="velocity"/>
             </joint>
-            <joint name="scoop_a">
-                <param name="node_id">0x5</param>
+            <joint name="servo_scoop_a">
+                <param name="node_id">0x3</param> <!-- 0x5 -->
                 <param name="gear_ratio">1</param>
                 <param name="max_pos">178</param> <!-- degrees -->
@@ -45,6 +45,6 @@
                 <state_interface name="position"/>
             </joint>
-            <joint name="scoop_b">
-                <param name="node_id">0x3</param>
+            <joint name="servo_scoop_b">
+                <param name="node_id">0x5</param> <!-- 0x3 -->
                 <param name="gear_ratio">1</param>
                 <param name="max_pos">178</param> <!-- degrees -->
@@ -55,5 +55,5 @@
                 <state_interface name="position"/>
             </joint>
-            <joint name="auger">
+            <joint name="servo_sampler_lift">
                 <param name="node_id">0x4</param>
                 <param name="gear_ratio">1</param>
@@ -67,6 +67,6 @@
                 <state_interface name="velocity"/>
             </joint>
-            <joint name="cap">
-                <param name="node_id">0x5</param>
+            <joint name="servo_cap">
+                <param name="node_id">0x6</param>
                 <param name="gear_ratio">1</param>
                 <param name="max_pos">270</param> <!-- degrees -->

File: src/description/ros2_control/science/science.talon.ros2_control.xacro (robot description, xacro)
@@ -10,5 +10,5 @@
         <param name="can_interface">can0</param>
       </hardware>
-      <joint name="talon_lift">
+      <joint name="talon_auger">
         <param name="node_id">1</param>
         <param name="joint_type">revolute</param>

Commit message: science now includes both sampler lift servos and cap servo has been renamed to auger lift

File: src/description/ros2_control/science/science.servo.ros2_control.xacro (robot description, xacro)
@@ -55,5 +55,5 @@
                 <state_interface name="position"/>
             </joint>
-            <joint name="servo_sampler_lift">
+            <joint name="servo_sampler_lift_l">
                 <param name="node_id">0x6</param>
                 <param name="gear_ratio">1</param>
@@ -67,5 +67,17 @@
                 <state_interface name="velocity"/>
             </joint>
-            <joint name="servo_cap">
+            <joint name="servo_sampler_lift_r">
+                <param name="node_id">0x0</param>
+                <param name="gear_ratio">1</param>
+                <param name="max_pos">90</param> <!-- degrees -->
+                <param name ="meters_per_deg">0.00016666666</param> <!-- (TODO) convert motor position in degrees to displacement in meters -->
+                <param name="servo_type">standard</param> <!-- standard / continuous -->
+                <param name="joint_type">prismatic</param> <!-- revolute / prismatic -->
+                <command_interface name="position"/>
+                <command_interface name="velocity"/>
+                <state_interface name="position"/>
+                <state_interface name="velocity"/>
+            </joint>
+            <joint name="servo_auger_lift">
                 <param name="node_id">0x4</param>
                 <param name="gear_ratio">1</param>

File: src/description/ros2_control/science/science.talon.ros2_control.xacro (robot description, xacro)
@@ -11,5 +11,5 @@
       </hardware>
       <joint name="talon_auger">
-        <param name="node_id">1</param>
+        <param name="node_id">2</param>
         <param name="joint_type">revolute</param>
         <!-- Motor config (goBilda Saturn 5303 Series 360 RPM) -->
