Commit message: fix: Use hex CAN IDs and add GPIO controller spawners

File: src/description/ros2_control/drive/drive.killswitch.ros2_control.xacro (robot description, xacro)
@@ -1,11 +1,10 @@
 <?xml version="1.0"?>
 <robot xmlns:xacro="http://www.ros.org/wiki/xacro">
-  <xacro:macro name="killswitch_ros2_control" params="name can_interface:=can0 can_id:=256">
-    <!-- CAN ID 0x100 = 256 decimal -->
+  <xacro:macro name="killswitch_ros2_control" params="name can_interface:=can0">
     <ros2_control name="${name}" type="system">
       <hardware>
         <plugin>killswitch_ros2_control/KillswitchHardwareInterface</plugin>
         <param name="can_interface">${can_interface}</param>
-        <param name="can_id">${can_id}</param>
+        <param name="can_id">0x100</param>
       </hardware>
       <gpio name="${name}">

File: src/description/ros2_control/science/science.laser.ros2_control.xacro (robot description, xacro)
@@ -1,11 +1,10 @@
 <?xml version="1.0"?>
 <robot xmlns:xacro="http://www.ros.org/wiki/xacro">
-    <xacro:macro name="laser_ros2_control" params="name can_interface:=can0 can_id:=304">
-        <!-- CAN ID 0x130 = 304 decimal -->
+    <xacro:macro name="laser_ros2_control" params="name can_interface:=can0">
         <ros2_control name="${name}" type="system">
             <hardware>
                 <plugin>laser_ros2_control/LaserHardwareInterface</plugin>
                 <param name="can_interface">${can_interface}</param>
-                <param name="can_id">${can_id}</param>
+                <param name="can_id">0x130</param>
             </hardware>
             <gpio name="${name}">
