Commit message: fixing rmd and smc hwis, real hardware should be good. fixed inconsistent naming convention in drive urdf. odrives having issues

File: src/description/ros2_control/drive/drive.odrive.ros2_control.xacro (robot description, xacro)
@@ -7,5 +7,5 @@
         <param name="can">can0</param>
       </hardware>
-      <joint name="swerve_module_front_left_joint">
+      <joint name="steer_fl_joint">
         <param name="node_id">6</param>
         <param name="gear_ratio">1</param>
@@ -17,5 +17,5 @@
         <state_interface name="velocity"/>
       </joint>
-      <joint name="swerve_module_front_right_joint">
+      <joint name="steer_fr_joint">
         <param name="node_id">5</param>
         <param name="gear_ratio">1</param>

File: src/description/ros2_control/drive/drive.rmd.ros2_control.xacro (robot description, xacro)
@@ -6,5 +6,5 @@
         <plugin>rmd_ros2_control/RMDHardwareInterface</plugin>
       </hardware>
-      <joint name="wheel_front_left_joint">
+      <joint name="propulsion_fl_joint">
         <param name="node_write_id">323</param> <!-- 0x143 -->
         <param name="node_read_id">579</param> <!-- 0x243 -->
@@ -18,5 +18,5 @@
         <state_interface name="velocity"/>
       </joint>
-      <joint name="wheel_front_right_joint">
+      <joint name="propulsion_fr_joint">
         <param name="node_write_id">322</param> <!-- 0x142 -->
         <param name="node_read_id">578</param> <!-- 0x242 -->
@@ -30,5 +30,5 @@
         <state_interface name="velocity"/>
       </joint>
-      <joint name="wheel_back_left_joint">
+      <joint name="propulsion_bl_joint">
         <param name="node_write_id">321</param> <!-- 0x141 -->
         <param name="node_read_id">577</param> <!-- 0x241 -->
@@ -42,5 +42,5 @@
         <state_interface name="velocity"/>
       </joint>
-      <joint name="wheel_back_right_joint">
+      <joint name="propulsion_br_joint">
         <param name="node_write_id">329</param> <!--0x149-->
         <param name="node_read_id">585</param> <!--0x249-->

File: src/description/urdf/athena_arm.urdf.xacro (robot description, xacro)
@@ -16,5 +16,5 @@
   <xacro:include filename="$(find description)/ros2_control/arm/arm.smc.ros2_control.xacro" />
   <!-- Import talon ros2_control description -->
-  <xacro:include filename="$(find description)/ros2_control/arm/arm.talon.ros2_control.xacro" />
+  <!-- <xacro:include filename="$(find description)/ros2_control/arm/arm.talon.ros2_control.xacro" /> -->
   <!-- Import rmd ros2_control description -->
   <xacro:include filename="$(find description)/ros2_control/arm/arm.rmd.ros2_control.xacro" />
@@ -32,5 +32,5 @@
   <xacro:unless value="$(arg use_mock_hardware)"> <!-- HARDWARE -->
     <xacro:smc_ros2_control name="smc"/>
-    <xacro:talon_ros2_control name="talon"/>
+    <!-- <xacro:talon_ros2_control name="talon"/> -->
     <xacro:rmd_ros2_control name="rmd"/>
     <xacro:actuator_ros2_control name="actuator"/>

File: src/description/urdf/athena_drive.urdf.xacro (robot description, xacro)
@@ -24,4 +24,7 @@
   <!-- Import odrive ros2_control description -->
   <xacro:include filename="$(find description)/ros2_control/drive/drive.odrive.ros2_control.xacro" />
+  <!-- create link fixed to the "world" -->
+  <link name="world"/>
+  <!-- Contains description of drive -->
   <xacro:description/>
   <xacro:if value="$(arg use_mock_hardware)">

File: src/description/urdf/athena_drive/athena_drive_macro.ros2_control.xacro (robot description, xacro)
@@ -42,5 +42,5 @@
     <state_interface name="velocity"/>
   </joint>
-  <joint name="${prefix}steer_1_joint">
+  <joint name="${prefix}steer_fl_joint">
     <command_interface name="position">
       <param name="min">0</param>
@@ -52,5 +52,5 @@
     <state_interface name="velocity"/>
   </joint>
-  <joint name="${prefix}steer_2_joint">
+  <joint name="${prefix}steer_fr_joint">
     <command_interface name="position">
       <param name="min">0</param>
@@ -62,5 +62,5 @@
     <state_interface name="velocity"/>
   </joint>
-  <joint name="${prefix}steer_3_joint">
+  <joint name="${prefix}steer_br_joint">
     <command_interface name="position">
       <param name="min">0</param>
@@ -72,5 +72,5 @@
     <state_interface name="velocity"/>
   </joint>
-  <joint name="${prefix}steer_4_joint">
+  <joint name="${prefix}steer_bl_joint">
     <command_interface name="position">
       <param name="min">0</param>
@@ -82,5 +82,5 @@
     <state_interface name="velocity"/>
   </joint>
-  <joint name="${prefix}propulsion_1_joint">
+  <joint name="${prefix}propulsion_fl_joint">
     <command_interface name="velocity"/>
     <state_interface name="position">
@@ -89,5 +89,5 @@
     <state_interface name="velocity"/>
   </joint>
-  <joint name="${prefix}propulsion_2_joint">
+  <joint name="${prefix}propulsion_fr_joint">
     <command_interface name="velocity"/>
     <state_interface name="position">
@@ -96,5 +96,5 @@
     <state_interface name="velocity"/>
   </joint>
-  <joint name="${prefix}propulsion_3_joint">
+  <joint name="${prefix}propulsion_br_joint">
     <state_interface name="position">
       <param name="initial_value">0.0</param>
@@ -102,5 +102,5 @@
     <state_interface name="velocity"/>
   </joint>
-  <joint name="${prefix}propulsion_4_joint">
+  <joint name="${prefix}propulsion_bl_joint">
     <state_interface name="position">
       <param name="initial_value">0.0</param>

File: src/description/urdf/athena_drive/athena_drive_macro.xacro (robot description, xacro)
@@ -181,5 +181,5 @@
     </joint>
     <!-- joint 2 -->
-    <joint name="${prefix}swerve_module_front_left_joint" type="revolute">
+    <joint name="${prefix}steer_fl_joint" type="revolute">
       <origin xyz="0 0 -0.3" rpy="${pi/2} 0 0"/>
       <parent link="${prefix}link1"/>
@@ -189,5 +189,5 @@
     </joint>
     <!-- joint 3 -->
-    <joint name="${prefix}wheel_front_left_joint" type="revolute">
+    <joint name="${prefix}propulsion_fl_joint" type="revolute">
       <origin xyz="0.8 0 0" rpy="0 0 0"/>
       <parent link="${prefix}link2"/>
@@ -205,5 +205,5 @@
     </joint>
     <!-- joint 5 -->
-    <joint name="${prefix}wheel_back_left_joint" type="revolute">
+    <joint name="${prefix}propulsion_bl_joint" type="revolute">
       <origin xyz="0 0 -0.15" rpy="0 ${pi/2} 0"/>
       <parent link="${prefix}link4"/>

File: src/description/urdf/athena_drive_description.urdf.xacro (robot description, xacro)
@@ -49,4 +49,11 @@
             </collision>
         </link>
+        <!-- base_joint fixes base_link to the environment -->
+        <joint name="base_joint" type="fixed">
+            <parent link="world"/>
+            <child link="chassis_base_link"/>
+            <origin xyz="0 0 0" rpy="0 0 3.141592653"/>
+            <axis xyz="0 0 1"/>
+        </joint>
         <joint name="suspension_front_left_joint" type="fixed">
             <origin xyz="0.61263 0.22146 -0.74592" rpy="1.5708 0 0.094743" />
@@ -106,5 +113,5 @@
             </collision>
         </link>
-        <joint name="steer_1_joint" type="revolute">
+        <joint name="steer_fl_joint" type="revolute">
             <origin xyz="0 0 0.059903" rpy="3.1416 0.094743 3.1416" />
             <parent link="swerve_mount_1_link" />
@@ -163,5 +170,5 @@
             </collision>
         </link>
-        <joint name="propulsion_1_joint" type="continuous">
+        <joint name="propulsion_fl_joint" type="continuous">
             <origin xyz="0 -0.054545 -0.10628" rpy="0 0 0" />
             <parent link="wheel_bracket_1_link" />
@@ -219,5 +226,5 @@
             </collision>
         </link>
-        <joint name="steer_4_joint" type="revolute">
+        <joint name="steer_bl_joint" type="revolute">
             <origin xyz="0 0 0.059903" rpy="0 -0.094743 0" />
             <parent link="swerve_mount_4_link" />
@@ -276,5 +283,5 @@
             </collision>
         </link>
-        <joint name="propulsion_4_joint" type="continuous">
+        <joint name="propulsion_bl_joint" type="continuous">
             <origin xyz="0 -0.054545 -0.10628" rpy="0 0 0" />
             <parent link="wheel_bracket_4_link" />
@@ -361,5 +368,5 @@
             </collision>
         </link>
-        <joint name="steer_2_joint" type="revolute">
+        <joint name="steer_fr_joint" type="revolute">
             <origin xyz="0 0 0.059903" rpy="3.1416 0.094743 3.1416" />
             <parent link="swerve_mount_2_link" />
@@ -418,5 +425,5 @@
             </collision>
         </link>
-        <joint name="propulsion_2_joint" type="continuous">
+        <joint name="propulsion_fr_joint" type="continuous">
             <origin xyz="0 -0.054545 -0.10628" rpy="0 0 0" />
             <parent link="wheel_bracket_2_link" />
@@ -474,5 +481,5 @@
             </collision>
         </link>
-        <joint name="steer_3_joint" type="revolute">
+        <joint name="steer_br_joint" type="revolute">
             <origin xyz="0 0 0.0599025014000917" rpy="0 -0.0947430505373176 0" />
             <parent link="swerve_mount_3_link" />
@@ -531,5 +538,5 @@
             </collision>
         </link>
-        <joint name="propulsion_3_joint" type="continuous">
+        <joint name="propulsion_br_joint" type="continuous">
             <origin xyz="0 -0.054545 -0.10628" rpy="0 0 0" />
             <parent link="wheel_bracket_3_link" />

Commit message: odrive upgrades

File: src/description/ros2_control/drive/drive.odrive.ros2_control.xacro (robot description, xacro)
@@ -1,9 +1,18 @@
 <?xml version="1.0"?>
 <robot xmlns:xacro="http://www.ros.org/wiki/xacro">
-  <xacro:macro name="odrive_ros2_control" params="name">
+  <xacro:macro name="odrive_ros2_control" params="name deactivate_odrive">
     <ros2_control name="${name}" type="system">
       <hardware>
-        <plugin>odrive_ros2_control_plugin/ODriveHardwareInterface</plugin>
-        <param name="can">can1</param>
+        <param name="deactivate_odrive">${deactivate_odrive}</param>
+        <xacro:if value="${deactivate_odrive}">
+          <plugin>mock_components/GenericSystem</plugin>
+        </xacro:if>
+        <xacro:unless value="${deactivate_odrive}">
+          <plugin>odrive_ros2_control_plugin/ODriveHardwareInterface</plugin>
+          <param name="update_rate">30</param> <!-- Hz -->
+          <param name="logger_rate">5</param> <!-- Hz -->
+          <param name="logger_state">0</param> <!-- 0 for off, 1 for on -->
+          <param name="can">can1</param>
+        </xacro:unless>
       </hardware>
       <joint name="steer_bl_joint">
@@ -12,8 +21,8 @@
         <command_interface name="position"/>
         <command_interface name="velocity"/>
-        <state_interface name="position">
-          <param name="initial_value">0.0</param>
-        </state_interface>
+        <state_interface name="position"/>
         <state_interface name="velocity"/>
+        <state_interface name="motor_temperature"/>
+        <state_interface name="torque_current"/>
       </joint>
       <joint name="steer_br_joint">
@@ -22,8 +31,8 @@
         <command_interface name="position"/>
         <command_interface name="velocity"/>
-        <state_interface name="position">
-          <param name="initial_value">0.0</param>
-        </state_interface>
+        <state_interface name="position"/>
         <state_interface name="velocity"/>
+        <state_interface name="motor_temperature"/>
+        <state_interface name="torque_current"/>
       </joint>
     </ros2_control>

File: src/description/urdf/athena_drive.urdf.xacro (robot description, xacro)
@@ -7,4 +7,5 @@
   <xacro:arg name="sim_gazebo" default="true"/>
   <xacro:arg name="simulation_controllers" default=""/>
+  <xacro:arg name="deactivate_odrive" default="false"/>
   <xacro:include filename="$(find description)/urdf/athena_drive/athena_drive_macro.xacro"/>
   <xacro:include filename="$(find description)/urdf/athena_drive/athena_drive_macro.ros2_control.xacro"/>
@@ -52,5 +53,7 @@
   </xacro:if>
   <xacro:unless value="$(arg use_mock_hardware)">
-    <xacro:odrive_ros2_control name="odrive"/>
+    <!-- ODrives-->
+    <xacro:odrive_ros2_control name="odrive" deactivate_odrive="$(arg deactivate_odrive)"/>
+    <!-- RMD -->
     <xacro:rmd_ros2_control name="rmd"/>
     <!-- LED status indicator (GPIO-based) -->
