Commit message: saving progress, killswitch seems to not be sending can messages for some reason

File: src/description/ros2_control/drive/drive.led.ros2_control.xacro (robot description, xacro)
@@ -7,4 +7,7 @@
         <param name="gpio_pin">${gpio_pin}</param>
         <param name="default_state">${default_state}</param>
+        <param name="update_rate">10</param> <!-- Hz -->
+        <param name="logger_rate">5</param> <!-- Hz -->
+        <param name="logger_state">0</param> <!-- 0 for off, 1 for on -->
       </hardware>
       <gpio name="${name}">

File: src/description/ros2_control/drive/drive.power_module.ros2_control.xacro (robot description, xacro)
@@ -1,10 +1,13 @@
 <?xml version="1.0"?>
 <robot xmlns:xacro="http://www.ros.org/wiki/xacro">
-  <xacro:macro name="killswitch_ros2_control" params="name can_interface:=can0">
+  <xacro:macro name="power_module_ros2_control" params="name can_interface:=can0">
     <ros2_control name="${name}" type="system">
       <hardware>
-        <plugin>killswitch_ros2_control/KillswitchHardwareInterface</plugin>
+        <plugin>power_module_ros2_control/PowerModuleHardwareInterface</plugin>
         <param name="can_interface">${can_interface}</param>
         <param name="can_id">0x100</param>
+        <param name="update_rate">10</param> <!-- Hz -->
+        <param name="logger_rate">5</param> <!-- Hz -->
+        <param name="logger_state">0</param> <!-- 0 for off, 1 for on -->
       </hardware>
       <gpio name="${name}">

File: src/description/ros2_control/science/science.laser.ros2_control.xacro (robot description, xacro)
@@ -7,4 +7,7 @@
                 <param name="can_interface">${can_interface}</param>
                 <param name="can_id">0x130</param>
+                <param name="update_rate">10</param> <!-- Hz -->
+                <param name="logger_rate">5</param> <!-- Hz -->
+                <param name="logger_state">0</param> <!-- 0 for off, 1 for on -->
             </hardware>
             <gpio name="${name}">

File: src/description/urdf/athena_drive.urdf.xacro (robot description, xacro)
@@ -29,6 +29,6 @@
   <!-- Import LED ros2_control description -->
   <xacro:include filename="$(find description)/ros2_control/drive/drive.led.ros2_control.xacro" />
-  <!-- Import killswitch ros2_control description -->
-  <xacro:include filename="$(find description)/ros2_control/drive/drive.killswitch.ros2_control.xacro" />
+  <!-- Import power_module ros2_control description -->
+  <xacro:include filename="$(find description)/ros2_control/drive/drive.power_module.ros2_control.xacro" />
   <!-- Contains description of drive -->
   <xacro:description/>
@@ -59,6 +59,6 @@
     <!-- LED status indicator (GPIO-based) -->
     <xacro:led_ros2_control name="status_led" gpio_pin="25"/>
-    <!-- Killswitch (CAN-based) -->
-    <xacro:killswitch_ros2_control name="drive_killswitch"/>
+    <!-- PowerModule (CAN-based) -->
+    <xacro:power_module_ros2_control name="drive_power_module"/>
   </xacro:unless>
 </robot>

Commit message: saving changes, for some reason I cant see power module can commands being sent

File: src/description/ros2_control/drive/drive.led.ros2_control.xacro (robot description, xacro)
@@ -1,10 +1,10 @@
 <?xml version="1.0"?>
 <robot xmlns:xacro="http://www.ros.org/wiki/xacro">
-  <xacro:macro name="led_ros2_control" params="name gpio_pin default_state:=off">
+  <xacro:macro name="led_ros2_control" params="name can_interface">
     <ros2_control name="${name}" type="system">
       <hardware>
         <plugin>led_ros2_control/LEDHardwareInterface</plugin>
-        <param name="gpio_pin">${gpio_pin}</param>
-        <param name="default_state">${default_state}</param>
+        <param name="can_interface">${can_interface}</param>
+        <param name="can_id">0x120</param>
         <param name="update_rate">10</param> <!-- Hz -->
         <param name="logger_rate">5</param> <!-- Hz -->
@@ -12,8 +12,10 @@
       </hardware>
       <gpio name="${name}">
-        <state_interface name="led_state"/>
-        <state_interface name="is_connected"/>
+        <param name="is_rgb">true</param>
         <state_interface name="status"/>
-        <command_interface name="led_command"/>
+        <command_interface name="red"/>
+        <command_interface name="green"/>
+        <command_interface name="blue"/>
+        <command_interface name="intensity"/>
         <command_interface name="status_request"/>
       </gpio>

File: src/description/ros2_control/drive/drive.power_module.ros2_control.xacro (robot description, xacro)
@@ -12,12 +12,13 @@
       </hardware>
       <gpio name="${name}">
+        <state_interface name="status"/>
         <state_interface name="kill_all_sent"/>
+        <state_interface name="kill_jetson_sent"/>
         <state_interface name="kill_main_sent"/>
-        <state_interface name="kill_jetson_sent"/>
-        <state_interface name="is_connected"/>
-        <state_interface name="status"/>
+        <state_interface name="kill_by_voltage_sent"/>
         <command_interface name="kill_all"/>
         <command_interface name="kill_main"/>
         <command_interface name="kill_jetson"/>
+        <command_interface name="kill_by_voltage"/>
         <command_interface name="status_request"/>
       </gpio>

File: src/description/urdf/athena_drive.urdf.xacro (robot description, xacro)
@@ -58,7 +58,7 @@
     <xacro:rmd_ros2_control name="rmd"/>
     <!-- LED status indicator (GPIO-based) -->
-    <xacro:led_ros2_control name="status_led" gpio_pin="25"/>
+    <xacro:led_ros2_control name="status_led" can_interface="can0"/>
     <!-- PowerModule (CAN-based) -->
-    <xacro:power_module_ros2_control name="drive_power_module"/>
+    <xacro:power_module_ros2_control name="drive_power_module" can_interface="can0"/>
   </xacro:unless>
 </robot>

Commit message: squash merged comp-science-upgrades

File: src/description/ros2_control/drive/drive.led.ros2_control.xacro (robot description, xacro)
@@ -12,7 +12,6 @@
       </hardware>
       <gpio name="${name}">
-        <param name="is_rgb">true</param>
         <param name="node_id">0</param>
-        <state_interface name="status"/>
+        <param name="mode">1</param> <!-- 0: intensity (0x20), 1: rgb (0x30), 2: toggle (0x40) -->
         <command_interface name="red"/>
         <command_interface name="green"/>
@@ -20,4 +19,5 @@
         <!-- <command_interface name="intensity"/> -->
         <command_interface name="status_request"/>
+        <state_interface name="status"/>
       </gpio>
     </ros2_control>

File: src/description/ros2_control/science/science.laser.ros2_control.xacro (robot description, xacro)
@@ -1,10 +1,10 @@
 <?xml version="1.0"?>
 <robot xmlns:xacro="http://www.ros.org/wiki/xacro">
-    <xacro:macro name="laser_ros2_control" params="name can_interface:=can0">
+    <xacro:macro name="laser_ros2_control" params="name can_interface:=can0 port_id:=0">
         <ros2_control name="${name}" type="system">
             <hardware>
                 <plugin>laser_ros2_control/LaserHardwareInterface</plugin>
                 <param name="can_interface">${can_interface}</param>
-                <param name="can_id">0x130</param>
+                <param name="can_id">0x100</param>
                 <param name="update_rate">10</param> <!-- Hz -->
                 <param name="logger_rate">5</param> <!-- Hz -->
@@ -12,4 +12,5 @@
             </hardware>
             <gpio name="${name}">
+                <param name="node_id">1</param>
                 <state_interface name="laser_state"/>
                 <state_interface name="temperature"/>

File: src/description/ros2_control/science/science.led.ros2_control.xacro (robot description, xacro)
@@ -12,9 +12,10 @@
       </hardware>
       <gpio name="fluoro_led">
-        <param name="is_rgb">false</param>
-        <param name="node_id">0</param>
+        <param name="node_id">1</param>
+        <param name="mode">2</param>
+        <command_interface name="toggle"/>
+        <command_interface name="status_request"/>
+        <state_interface name="is_connected"/>
         <state_interface name="status"/>
-        <command_interface name="intensity"/>
-        <command_interface name="status_request"/>
       </gpio>
     </ros2_control>

File: src/description/ros2_control/science/science.limit_switch.ros2_control.xacro (robot description, xacro)
@@ -16,4 +16,9 @@
         <command_interface name="status_request"/>
       </gpio>
+      <gpio name="science_magnetic_limit_switch">
+        <param name="node_id">1</param>
+        <state_interface name="status"/>
+        <command_interface name="status_request"/>
+      </gpio>
     </ros2_control>
   </xacro:macro>

File: src/description/urdf/athena_drive.urdf.xacro (robot description, xacro)
@@ -32,4 +32,6 @@
   <!-- Import power_module ros2_control description -->
   <xacro:include filename="$(find description)/ros2_control/drive/drive.power_module.ros2_control.xacro" />
+  <!-- Added servo_drive here -->
+  <xacro:include filename="$(find description)/ros2_control/drive/drive.servo.ros2_control.xacro"/>
   <!-- Contains description of drive -->
   <xacro:description/>
@@ -62,4 +64,6 @@
     <!-- PowerModule (CAN-based) -->
     <xacro:power_module_ros2_control name="drive_power_module" can_interface="$(arg can_interface)"/>
+    <!-- Servo control for Zed camera -->
+    <xacro:servo_ros2_control name="zed_servo_control" can_interface="$(arg can_interface)"/>
   </xacro:unless>
 </robot>

File: src/description/urdf/athena_science.urdf.xacro (robot description, xacro)
@@ -11,6 +11,9 @@
   <xacro:include filename="$(find description)/ros2_control/science/science.talon.ros2_control.xacro"/>
   <xacro:include filename="$(find description)/ros2_control/science/science.laser.ros2_control.xacro"/>
+  <xacro:include filename="$(find description)/ros2_control/science/science.ccd.ros2_control.xacro"/>
+  <xacro:include filename="$(find description)/ros2_control/science/science.photodiode.ros2_control.xacro"/>
   <xacro:include filename="$(find description)/ros2_control/science/science.led.ros2_control.xacro"/>
   <xacro:include filename="$(find description)/ros2_control/science/science.limit_switch.ros2_control.xacro"/>
+  <xacro:include filename="$(find description)/ros2_control/science/science.rotary_encoder.ros2_control.xacro"/>
   <!-- create link fixed to the "world" -->
   <link name="world"/>
@@ -32,7 +35,12 @@
     <!-- Import laser ros2_control description (CAN-based) -->
     <xacro:laser_ros2_control name="spectrometry_laser" can_interface="$(arg can_interface)"/>
-    <!-- Import LED and limit switch ros2_control descriptions -->
+    <!-- Import CCD ros2_control description (CAN-based) -->
+    <xacro:ccd_ros2_control name="spectrometry_ccd" can_interface="$(arg can_interface)"/>
+    <!-- Import photodiode ros2_control description (CAN-based) -->
+    <xacro:photodiode_ros2_control name="photodiode" can_interface="$(arg can_interface)"/>
+    <!-- Import LED, limit switch, and rotary encoder ros2_control descriptions -->
     <xacro:science_led_ros2_control name="fluoro_led_hwi" can_interface="$(arg can_interface)"/>
     <xacro:science_limit_switch_ros2_control name="science_limit_switch_hwi" can_interface="$(arg can_interface)"/>
+    <xacro:science_rotary_encoder_ros2_control name="science_rotary_encoder_hwi" can_interface="$(arg can_interface)"/>
   </xacro:unless>
 </robot>
