Commit message: working robot

File: src/description/ros2_control/arm/arm.rmd.ros2_control.xacro (robot description, xacro)
@@ -11,5 +11,5 @@
       </hardware>
       <joint name="shoulder_pitch">
-        <param name="node_id">0x14A</param>
+        <param name="node_id">0x149</param>
         <param name="gear_ratio">100</param>
         <param name="joint_orientation">1.0</param>
@@ -26,4 +26,12 @@
         <state_interface name="velocity"/>
       </joint>
+      <joint name="gripper_claw">
+        <param name="node_id">0x169</param>
+        <param name="gear_ratio">100</param>
+        <param name="joint_orientation">1.0</param>
+        <param name="operating_velocity">150</param> <!-- motor dps -->
+        <state_interface name="position"/>
+        <state_interface name="velocity"/>
+      </joint>
     </ros2_control>
   </xacro:macro>

File: src/description/ros2_control/drive/drive.odrive.ros2_control.xacro (robot description, xacro)
@@ -8,6 +8,6 @@
       </hardware>
       <joint name="steer_fl_joint">
-        <param name="node_id">6</param>
-        <param name="gear_ratio">10</param>
+        <param name="node_id">5</param>
+        <param name="gear_ratio">26</param>
         <command_interface name="position"/>
         <command_interface name="velocity"/>
@@ -18,6 +18,6 @@
       </joint>
       <joint name="steer_fr_joint">
-        <param name="node_id">5</param>
-        <param name="gear_ratio">10</param>
+        <param name="node_id">6</param>
+        <param name="gear_ratio">26</param>
         <command_interface name="position"/>
         <command_interface name="velocity"/>

File: src/description/ros2_control/drive/drive.rmd.ros2_control.xacro (robot description, xacro)
@@ -5,5 +5,5 @@
       <hardware>
         <plugin>rmd_ros2_control/RMDHardwareInterface</plugin>
-        <param name="update_rate">10</param> <!-- Hz -->
+        <param name="update_rate">30</param> <!-- Hz -->
         <param name="logger_rate">5</param> <!-- Hz -->
         <param name="logger_state">0</param> <!-- 0 for off, 1 for on -->

File: src/description/urdf/athena_arm.urdf.xacro (robot description, xacro)
@@ -16,5 +16,5 @@
   <xacro:include filename="$(find description)/ros2_control/arm/arm.smc.ros2_control.xacro" />
   <!-- Import talon ros2_control description -->
-  <xacro:include filename="$(find description)/ros2_control/arm/arm.talon.ros2_control.xacro" />
+  <!-- <xacro:include filename="$(find description)/ros2_control/arm/arm.talon.ros2_control.xacro" /> -->
   <!-- Import rmd ros2_control description -->
   <xacro:include filename="$(find description)/ros2_control/arm/arm.rmd.ros2_control.xacro" />
@@ -32,5 +32,5 @@
   <xacro:unless value="$(arg use_mock_hardware)"> <!-- HARDWARE -->
     <xacro:smc_ros2_control name="smc"/>
-    <xacro:talon_ros2_control name="talon"/>
+    <!-- <xacro:talon_ros2_control name="talon"/> -->
     <xacro:rmd_ros2_control name="rmd"/>
     <xacro:servo_ros2_control name="servo"/>
