Commit message: working, but code wise it should not be prismatic, suitable for now

File: src/description/ros2_control/arm/arm.talon_3dof.ros2_control.xacro (robot description, xacro)
@@ -7,28 +7,9 @@
         <param name="update_rate">10</param> <!-- Hz -->
         <param name="logger_rate">5</param> <!-- Hz -->
-        <param name="logger_state">0</param> <!-- 0 for off, 1 for on -->
+        <param name="logger_state">1</param> <!-- 0 for off, 1 for on -->
         <param name="can_interface">can0</param>
       </hardware>
-      <joint name="gripper_claw">
-        <param name="node_id">2</param>
-        <param name="max_disp">0.06</param> <!-- meters -->
-        <param name="joint_type">prismatic</param>
-        <!-- Motor config (Pololu 37D defaults) -->
-        <param name="encoder_resolution">64.0</param>
-        <param name="gear_ratio">102.08</param>
-        <param name="distance_per_rev">0.0015</param> <!-- m/rev -->
-        <param name="inverted">true</param>
-        <param name="sensor_phase">true</param>
-        <param name="kP">0.25</param>
-        <param name="kI">0.0</param>
-        <param name="kD">0.0</param>
-        <param name="kF">0.0</param>
-        <command_interface name="position"/>
-        <command_interface name="velocity"/>
-        <state_interface name="position"/>
-        <state_interface name="velocity"/>
-      </joint>
       <joint name="wrist_motor_a">
-        <param name="node_id">3</param>
+        <param name="node_id">6</param>
         <param name="max_disp">0.06</param> <!-- meters -->
         <param name="joint_type">prismatic</param>
@@ -86,4 +67,23 @@
         <state_interface name="velocity"/>
       </joint>
+      <joint name="gripper_claw">
+        <param name="node_id">2</param>
+        <param name="max_disp">0.06</param> <!-- meters -->
+        <param name="joint_type">prismatic</param>
+        <!-- Motor config (Pololu 37D defaults) -->
+        <param name="encoder_resolution">64.0</param>
+        <param name="gear_ratio">102.08</param>
+        <param name="distance_per_rev">0.0015</param> <!-- m/rev -->
+        <param name="inverted">true</param>
+        <param name="sensor_phase">true</param>
+        <param name="kP">0.25</param>
+        <param name="kI">0.0</param>
+        <param name="kD">0.0</param>
+        <param name="kF">0.0</param>
+        <command_interface name="position"/>
+        <command_interface name="velocity"/>
+        <state_interface name="position"/>
+        <state_interface name="velocity"/>
+      </joint>
     </ros2_control>
   </xacro:macro>
