Commit message: allows the user to deactivate the talons and have a mock hardware replacement for just those joints

File: src/description/ros2_control/arm/arm.talon_2dof.ros2_control.xacro (robot description, xacro)
@@ -1,12 +1,18 @@
 <?xml version="1.0"?>
 <robot xmlns:xacro="http://www.ros.org/wiki/xacro">
-  <xacro:macro name="talon_2dof_ros2_control" params="name">
+  <xacro:macro name="talon_2dof_ros2_control" params="name deactivate_talon">
     <ros2_control name="${name}" type="system">
       <hardware>
-        <plugin>talon_ros2_control/TALONHardwareInterface</plugin>
-        <param name="update_rate">10</param> <!-- Hz -->
-        <param name="logger_rate">5</param> <!-- Hz -->
-        <param name="logger_state">0</param> <!-- 0 for off, 1 for on -->
-        <param name="can_interface">can0</param>
+        <param name="deactivate_talon">${deactivate_talon}</param>
+        <xacro:if value="${deactivate_talon}">
+          <plugin>mock_components/GenericSystem</plugin>
+        </xacro:if>
+        <xacro:unless value="${deactivate_talon}">
+          <plugin>talon_ros2_control/TALONHardwareInterface</plugin>
+          <param name="update_rate">10</param> <!-- Hz -->
+          <param name="logger_rate">5</param> <!-- Hz -->
+          <param name="logger_state">0</param> <!-- 0 for off, 1 for on -->
+          <param name="can_interface">can0</param>
+        </xacro:unless>
       </hardware>
       <joint name="gripper_claw">

File: src/description/ros2_control/arm/arm.talon_3dof.ros2_control.xacro (robot description, xacro)
@@ -1,12 +1,17 @@
 <?xml version="1.0"?>
 <robot xmlns:xacro="http://www.ros.org/wiki/xacro">
-  <xacro:macro name="talon_3dof_ros2_control" params="name">
+  <xacro:macro name="talon_3dof_ros2_control" params="name deactivate_talon">
     <ros2_control name="${name}" type="system">
       <hardware>
-        <plugin>talon_ros2_control/TALONHardwareInterface</plugin>
-        <param name="update_rate">10</param> <!-- Hz -->
-        <param name="logger_rate">5</param> <!-- Hz -->
-        <param name="logger_state">1</param> <!-- 0 for off, 1 for on -->
-        <param name="can_interface">can0</param>
+        <xacro:if value="${deactivate_talon}">
+          <plugin>mock_components/GenericSystem</plugin>
+        </xacro:if>
+        <xacro:unless value="${deactivate_talon}">
+          <plugin>talon_ros2_control/TALONHardwareInterface</plugin>
+          <param name="update_rate">10</param> <!-- Hz -->
+          <param name="logger_rate">5</param> <!-- Hz -->
+          <param name="logger_state">0</param> <!-- 0 for off, 1 for on -->
+          <param name="can_interface">can0</param>
+        </xacro:unless>
       </hardware>
       <joint name="wrist_motor_a">

File: src/description/urdf/athena_arm.urdf.xacro (robot description, xacro)
@@ -9,4 +9,5 @@
   <xacro:arg name="simulation_controllers" default=""/>
   <xacro:arg name="use_3dof" default="false"/>
+  <xacro:arg name="deactivate_talon" default="false"/>
   <!-- Macro Imports -->
   <!-- Import athena_arm macro -->
@@ -35,9 +36,9 @@
   <xacro:unless value="$(arg use_mock_hardware)"> <!-- HARDWARE -->
     <xacro:if value="$(arg use_3dof)">
-      <xacro:talon_3dof_ros2_control name="talon"/>
+      <xacro:talon_3dof_ros2_control name="talon" deactivate_talon="$(arg deactivate_talon)"/>
       <xacro:smc_3dof_ros2_control name="smc"/>
     </xacro:if>
     <xacro:unless value="$(arg use_3dof)">
-      <xacro:talon_2dof_ros2_control name="talon"/>
+      <xacro:talon_2dof_ros2_control name="talon" deactivate_talon="$(arg deactivate_talon)"/>
       <xacro:smc_2dof_ros2_control name="smc"/>
     </xacro:unless>
