Commit message: added limit switch and rotary encoder HWI, included all necessary HWIs, needs fixing

File: src/description/ros2_control/arm/arm.servo.ros2_control.xacro (robot description, xacro)
@@ -29,4 +29,38 @@
                 <state_interface name="status"/>
             </joint>
+            <joint name="cam_0">
+                <param name="node_id">0x2</param>
+                <param name="gear_ratio">1</param>
+                <param name="max_pos">180</param> <!-- degrees -->
+                <param name="servo_type">standard</param> <!-- standard or continuous -->
+                <param name="joint_type">revolute</param> <!-- revolute or prismatic -->
+                <command_interface name="position" />
+                <command_interface name="velocity"/>
+                <command_interface name="status_request"/>
+                <command_interface name="maintenance_request"/>
+                <command_interface name="maintenance_frame_high"/>
+                <command_interface name="maintenance_frame_low"/>
+                <command_interface name="maintenance_data_count"/>
+                <state_interface name="position"/>
+                <state_interface name="velocity"/>
+                <state_interface name="status"/>
+            </joint>
+            <joint name="cam_1">
+                <param name="node_id">0x3</param>
+                <param name="gear_ratio">1</param>
+                <param name="max_pos">180</param> <!-- degrees -->
+                <param name="servo_type">standard</param> <!-- standard or continuous -->
+                <param name="joint_type">revolute</param> <!-- revolute or prismatic -->
+                <command_interface name="position" />
+                <command_interface name="velocity"/>
+                <command_interface name="status_request"/>
+                <command_interface name="maintenance_request"/>
+                <command_interface name="maintenance_frame_high"/>
+                <command_interface name="maintenance_frame_low"/>
+                <command_interface name="maintenance_data_count"/>
+                <state_interface name="position"/>
+                <state_interface name="velocity"/>
+                <state_interface name="status"/>
+            </joint>
         </ros2_control>
     </xacro:macro>

File: src/description/ros2_control/science/science.servo.ros2_control.xacro (robot description, xacro)
@@ -7,5 +7,5 @@
                 <param name="update_rate">20</param> <!-- Hz -->
                 <param name="logger_rate">5</param> <!-- Hz -->
-                <param name="logger_state">1</param> <!-- 0 for off, 1 for on -->
+                <param name="logger_state">0</param> <!-- 0 for off, 1 for on -->
                 <param name="can_interface">can0</param>
                 <param name="can_id">0x80</param>

File: src/description/urdf/athena_science.urdf.xacro (robot description, xacro)
@@ -9,4 +9,6 @@
   <xacro:include filename="$(find description)/ros2_control/science/science.talon.ros2_control.xacro"/>
   <xacro:include filename="$(find description)/ros2_control/science/science.laser.ros2_control.xacro"/>
+  <xacro:include filename="$(find description)/ros2_control/science/science.led.ros2_control.xacro"/>
+  <xacro:include filename="$(find description)/ros2_control/science/science.limit_switch.ros2_control.xacro"/>
   <!-- create link fixed to the "world" -->
   <link name="world"/>
@@ -26,4 +28,7 @@
     <!-- Import laser ros2_control description (CAN-based) -->
     <xacro:laser_ros2_control name="spectrometry_laser"/>
+    <!-- Import LED and limit switch ros2_control descriptions -->
+    <xacro:science_led_ros2_control name="fluoro_led_hwi"/>
+    <xacro:science_limit_switch_ros2_control name="science_limit_switch_hwi"/>
   </xacro:unless>
 </robot>
