Commit message: Add equipment servicing functionality

File: src/description/ros2_control/arm/arm.base_limit_switch.ros2_control.xacro (robot description, xacro)
@@ -7,5 +7,5 @@
         <param name="can_interface">${can_interface}</param>
         <param name="can_id">0x130</param>
-        <param name="update_rate">2</param>
+        <param name="update_rate">0</param>
         <param name="logger_rate">5</param>
         <param name="logger_state">0</param>

File: src/description/ros2_control/arm/arm.rotary_encoder.ros2_control.xacro (robot description, xacro)
@@ -7,5 +7,5 @@
         <param name="can_interface">${can_interface}</param>
         <param name="can_id">0x130</param>
-        <param name="update_rate">2</param>
+        <param name="update_rate">0</param>
         <param name="logger_rate">5</param>
         <param name="logger_state">0</param>

File: src/description/ros2_control/arm/arm.servo.ros2_control.xacro (robot description, xacro)
@@ -5,5 +5,5 @@
             <hardware>
                 <plugin>servo_ros2_control/SERVOHardwareInterface</plugin>
-                <param name="update_rate">1</param> <!-- Hz -->
+                <param name="update_rate">0</param> <!-- Hz -->
                 <param name="logger_rate">5</param> <!-- Hz -->
                 <param name="logger_state">0</param> <!-- 0 for off, 1 for on -->

File: src/description/ros2_control/arm/arm.smc_2dof.ros2_control.xacro (robot description, xacro)
@@ -28,9 +28,9 @@
         <state_interface name="status"/>
       </joint>
-      <joint name="wrist_pitch">
+      <!-- <joint name="wrist_pitch">
         <param name="node_id">0x147</param>
         <param name="gear_ratio">40</param>
         <param name="joint_orientation">1.0</param>
-        <param name="operating_velocity">1000</param> <!-- motor dps -->
+        <param name="operating_velocity">1000</param> <!- motor dps ->
         <command_interface name="position"/>
         <command_interface name="velocity"/>
@@ -45,5 +45,5 @@
         <state_interface name="torque_current"/>
         <state_interface name="status"/>
-      </joint>
+      </joint> -->
       <joint name="wrist_roll">
         <param name="node_id">0x145</param>

File: src/description/ros2_control/arm/arm.talon_2dof.ros2_control.xacro (robot description, xacro)
@@ -16,4 +16,43 @@
         </xacro:unless>
       </hardware>
+      <joint name="wrist_pitch">
+        <param name="node_id">0</param>
+        <param name="joint_type">revolute</param>
+        <!-- Motor config (Pololu 37D defaults) -->
+        <param name="encoder_resolution">64.0</param>
+        <param name="gear_ratio">4002.08</param>
+        <param name="inverted">true</param>
+        <param name="sensor_phase">true</param>
+        <param name="kP">0.25</param>
+        <param name="kI">0.0</param>
+        <param name="kD">0.0</param>
+        <param name="kF">0.0</param>
+        <param name="status_1_general_period_ms">255</param>
+        <param name="status_2_feedback0_period_ms">255</param>
+        <param name="status_3_quadrature_period_ms">255</param>
+        <param name="status_4_aintempvbat_period_ms">255</param>
+        <param name="status_6_misc_period_ms">255</param>
+        <param name="status_7_commstatus_period_ms">255</param>
+        <param name="status_8_pulsewidth_period_ms">255</param>
+        <param name="status_9_motprofbuffer_period_ms">255</param>
+        <param name="status_10_targets_period_ms">255</param>
+        <param name="status_12_feedback1_period_ms">255</param>
+        <param name="status_13_base_pidf0_period_ms">255</param>
+        <param name="status_14_turn_pidf1_period_ms">255</param>
+        <param name="status_15_firmwareapistatus_period_ms">255</param>
+        <param name="status_17_targets1_period_ms">255</param>
+        <param name="control_3_general_period_ms">50</param>
+        <param name="control_4_advanced_period_ms">255</param>
+        <param name="control_6_motprofaddtrajpoint_period_ms">255</param>
+        <param name="status_frame_timeout_ms">255</param>
+        <command_interface name="position"/>
+        <command_interface name="velocity"/>
+        <command_interface name="status_request"/>
+        <state_interface name="position"/>
+        <state_interface name="velocity"/>
+        <state_interface name="motor_temperature"/>
+        <state_interface name="torque_current"/>
+        <state_interface name="status"/>
+      </joint>
       <joint name="gripper_claw">
         <param name="node_id">4</param>
@@ -30,4 +69,22 @@
         <param name="kD">0.0</param>
         <param name="kF">0.0</param>
+        <param name="status_1_general_period_ms">255</param>
+        <param name="status_2_feedback0_period_ms">255</param>
+        <param name="status_3_quadrature_period_ms">255</param>
+        <param name="status_4_aintempvbat_period_ms">255</param>
+        <param name="status_6_misc_period_ms">255</param>
+        <param name="status_7_commstatus_period_ms">255</param>
+        <param name="status_8_pulsewidth_period_ms">255</param>
+        <param name="status_9_motprofbuffer_period_ms">255</param>
+        <param name="status_10_targets_period_ms">255</param>
+        <param name="status_12_feedback1_period_ms">255</param>
+        <param name="status_13_base_pidf0_period_ms">255</param>
+        <param name="status_14_turn_pidf1_period_ms">255</param>
+        <param name="status_15_firmwareapistatus_period_ms">255</param>
+        <param name="status_17_targets1_period_ms">255</param>
+        <param name="control_3_general_period_ms">50</param>
+        <param name="control_4_advanced_period_ms">255</param>
+        <param name="control_6_motprofaddtrajpoint_period_ms">255</param>
+        <param name="status_frame_timeout_ms">255</param>
         <command_interface name="position"/>
         <command_interface name="velocity"/>

File: src/description/ros2_control/arm/arm.talon_3dof.ros2_control.xacro (robot description, xacro)
@@ -28,4 +28,22 @@
         <param name="kD">0.0</param>
         <param name="kF">0.0</param>
+        <param name="status_1_general_period_ms">100</param>
+        <param name="status_2_feedback0_period_ms">20</param>
+        <param name="status_3_quadrature_period_ms">255</param>
+        <param name="status_4_aintempvbat_period_ms">100</param>
+        <param name="status_6_misc_period_ms">255</param>
+        <param name="status_7_commstatus_period_ms">255</param>
+        <param name="status_8_pulsewidth_period_ms">255</param>
+        <param name="status_9_motprofbuffer_period_ms">255</param>
+        <param name="status_10_targets_period_ms">255</param>
+        <param name="status_12_feedback1_period_ms">255</param>
+        <param name="status_13_base_pidf0_period_ms">255</param>
+        <param name="status_14_turn_pidf1_period_ms">255</param>
+        <param name="status_15_firmwareapistatus_period_ms">255</param>
+        <param name="status_17_targets1_period_ms">255</param>
+        <param name="control_3_general_period_ms">50</param>
+        <param name="control_4_advanced_period_ms">255</param>
+        <param name="control_6_motprofaddtrajpoint_period_ms">255</param>
+        <param name="status_frame_timeout_ms">100</param>
         <command_interface name="position"/>
         <command_interface name="velocity"/>
@@ -50,4 +68,22 @@
         <param name="kD">0.0</param>
         <param name="kF">0.0</param>
+        <param name="status_1_general_period_ms">100</param>
+        <param name="status_2_feedback0_period_ms">20</param>
+        <param name="status_3_quadrature_period_ms">255</param>
+        <param name="status_4_aintempvbat_period_ms">100</param>
+        <param name="status_6_misc_period_ms">255</param>
+        <param name="status_7_commstatus_period_ms">255</param>
+        <param name="status_8_pulsewidth_period_ms">255</param>
+        <param name="status_9_motprofbuffer_period_ms">255</param>
+        <param name="status_10_targets_period_ms">255</param>
+        <param name="status_12_feedback1_period_ms">255</param>
+        <param name="status_13_base_pidf0_period_ms">255</param>
+        <param name="status_14_turn_pidf1_period_ms">255</param>
+        <param name="status_15_firmwareapistatus_period_ms">255</param>
+        <param name="status_17_targets1_period_ms">255</param>
+        <param name="control_3_general_period_ms">50</param>
+        <param name="control_4_advanced_period_ms">255</param>
+        <param name="control_6_motprofaddtrajpoint_period_ms">255</param>
+        <param name="status_frame_timeout_ms">100</param>
         <command_interface name="position"/>
         <command_interface name="velocity"/>
@@ -72,4 +108,22 @@
         <param name="kD">0.0</param>
         <param name="kF">0.0</param>
+        <param name="status_1_general_period_ms">100</param>
+        <param name="status_2_feedback0_period_ms">20</param>
+        <param name="status_3_quadrature_period_ms">255</param>
+        <param name="status_4_aintempvbat_period_ms">100</param>
+        <param name="status_6_misc_period_ms">255</param>
+        <param name="status_7_commstatus_period_ms">255</param>
+        <param name="status_8_pulsewidth_period_ms">255</param>
+        <param name="status_9_motprofbuffer_period_ms">255</param>
+        <param name="status_10_targets_period_ms">255</param>
+        <param name="status_12_feedback1_period_ms">255</param>
+        <param name="status_13_base_pidf0_period_ms">255</param>
+        <param name="status_14_turn_pidf1_period_ms">255</param>
+        <param name="status_15_firmwareapistatus_period_ms">255</param>
+        <param name="status_17_targets1_period_ms">255</param>
+        <param name="control_3_general_period_ms">50</param>
+        <param name="control_4_advanced_period_ms">255</param>
+        <param name="control_6_motprofaddtrajpoint_period_ms">255</param>
+        <param name="status_frame_timeout_ms">100</param>
         <command_interface name="position"/>
         <command_interface name="velocity"/>
@@ -95,4 +149,22 @@
         <param name="kD">0.0</param>
         <param name="kF">0.0</param>
+        <param name="status_1_general_period_ms">100</param>
+        <param name="status_2_feedback0_period_ms">20</param>
+        <param name="status_3_quadrature_period_ms">255</param>
+        <param name="status_4_aintempvbat_period_ms">100</param>
+        <param name="status_6_misc_period_ms">255</param>
+        <param name="status_7_commstatus_period_ms">255</param>
+        <param name="status_8_pulsewidth_period_ms">255</param>
+        <param name="status_9_motprofbuffer_period_ms">255</param>
+        <param name="status_10_targets_period_ms">255</param>
+        <param name="status_12_feedback1_period_ms">255</param>
+        <param name="status_13_base_pidf0_period_ms">255</param>
+        <param name="status_14_turn_pidf1_period_ms">255</param>
+        <param name="status_15_firmwareapistatus_period_ms">255</param>
+        <param name="status_17_targets1_period_ms">255</param>
+        <param name="control_3_general_period_ms">50</param>
+        <param name="control_4_advanced_period_ms">255</param>
+        <param name="control_6_motprofaddtrajpoint_period_ms">255</param>
+        <param name="status_frame_timeout_ms">100</param>
         <command_interface name="position"/>
         <command_interface name="velocity"/>
