Commit message: Refactor robot stack to single use_sim launch argument

File: src/description/config/odrive.ros2_control.xacro (robot description, xacro)
@@ -1,9 +1,9 @@
 <?xml version="1.0"?>
 <robot xmlns:xacro="http://www.ros.org/wiki/xacro">
-  <xacro:macro name="odrive_ros2_control" params="name">
+  <xacro:macro name="odrive_ros2_control" params="name can_interface">
     <ros2_control name="${name}" type="system">
       <hardware>
         <plugin>odrive_ros2_control_plugin/ODriveHardwareInterface</plugin>
-        <param name="can">can0</param>
+        <param name="can_interface">${can_interface}</param>
       </hardware>
        <!--

File: src/description/ros2_control/arm/arm.rmd.ros2_control.xacro (robot description, xacro)
@@ -1,5 +1,5 @@
 <?xml version="1.0"?>
 <robot xmlns:xacro="http://www.ros.org/wiki/xacro">
-  <xacro:macro name="rmd_ros2_control" params="name">
+  <xacro:macro name="rmd_ros2_control" params="name can_interface">
     <ros2_control name="${name}" type="system">
       <hardware>
@@ -8,5 +8,5 @@
         <param name="logger_rate">5</param> <!-- Hz -->
         <param name="logger_state">0</param> <!-- 0 for off, 1 for on -->
-        <param name="can_interface">can0</param>
+        <param name="can_interface">${can_interface}</param>
       </hardware>
       <joint name="shoulder_pitch">

File: src/description/ros2_control/arm/arm.servo.ros2_control.xacro (robot description, xacro)
@@ -1,5 +1,5 @@
 <?xml version="1.0"?>
 <robot xmlns:xacro="http://www.ros.org/wiki/xacro">
-    <xacro:macro name="servo_ros2_control" params="name">
+    <xacro:macro name="servo_ros2_control" params="name can_interface">
         <ros2_control name="${name}" type="system">
             <hardware>
@@ -8,5 +8,5 @@
                 <param name="logger_rate">5</param> <!-- Hz -->
                 <param name="logger_state">0</param> <!-- 0 for off, 1 for on -->
-                <param name="can_interface">can0</param>
+                <param name="can_interface">${can_interface}</param>
                 <param name="can_id">0x80</param>
             </hardware>

File: src/description/ros2_control/arm/arm.smc.ros2_control.xacro (robot description, xacro)
@@ -1,5 +1,5 @@
 <?xml version="1.0"?>
 <robot xmlns:xacro="http://www.ros.org/wiki/xacro">
-  <xacro:macro name="smc_ros2_control" params="name">
+  <xacro:macro name="smc_ros2_control" params="name can_interface">
     <ros2_control name="${name}" type="system">
       <hardware>
@@ -8,5 +8,5 @@
         <param name="logger_rate">5</param> <!-- Hz -->
         <param name="logger_state">0</param> <!-- 0 for off, 1 for on -->
-        <param name="can_interface">can0</param>
+        <param name="can_interface">${can_interface}</param>
       </hardware>
       <joint name="base_yaw">

File: src/description/ros2_control/arm/arm.talon.ros2_control.xacro (robot description, xacro)
@@ -1,5 +1,5 @@
 <?xml version="1.0"?>
 <robot xmlns:xacro="http://www.ros.org/wiki/xacro">
-  <xacro:macro name="talon_ros2_control" params="name">
+  <xacro:macro name="talon_ros2_control" params="name can_interface">
     <ros2_control name="${name}" type="system">
       <hardware>
@@ -8,5 +8,5 @@
         <param name="logger_rate">5</param> <!-- Hz -->
         <param name="logger_state">0</param> <!-- 0 for off, 1 for on -->
-        <param name="can_interface">can0</param>
+        <param name="can_interface">${can_interface}</param>
       </hardware>
       <joint name="gripper_claw">

File: src/description/ros2_control/drive/drive.killswitch.ros2_control.xacro (robot description, xacro)
@@ -1,5 +1,5 @@
 <?xml version="1.0"?>
 <robot xmlns:xacro="http://www.ros.org/wiki/xacro">
-  <xacro:macro name="killswitch_ros2_control" params="name can_interface:=can0">
+  <xacro:macro name="killswitch_ros2_control" params="name can_interface">
     <ros2_control name="${name}" type="system">
       <hardware>

File: src/description/ros2_control/drive/drive.odrive.ros2_control.xacro (robot description, xacro)
@@ -1,9 +1,9 @@
 <?xml version="1.0"?>
 <robot xmlns:xacro="http://www.ros.org/wiki/xacro">
-  <xacro:macro name="odrive_ros2_control" params="name">
+  <xacro:macro name="odrive_ros2_control" params="name can_interface">
     <ros2_control name="${name}" type="system">
       <hardware>
         <plugin>odrive_ros2_control_plugin/ODriveHardwareInterface</plugin>
-        <param name="can">can0</param>
+        <param name="can_interface">${can_interface}</param>
       </hardware>
       <joint name="steer_bl_joint">

File: src/description/ros2_control/drive/drive.rmd.ros2_control.xacro (robot description, xacro)
@@ -1,5 +1,5 @@
 <?xml version="1.0"?>
 <robot xmlns:xacro="http://www.ros.org/wiki/xacro">
-  <xacro:macro name="rmd_ros2_control" params="name">
+  <xacro:macro name="rmd_ros2_control" params="name can_interface">
     <ros2_control name="${name}" type="system">
       <hardware>
@@ -8,5 +8,5 @@
         <param name="logger_rate">5</param> <!-- Hz -->
         <param name="logger_state">0</param> <!-- 0 for off, 1 for on -->
-        <param name="can_interface">can0</param>
+        <param name="can_interface">${can_interface}</param>
       </hardware>
       <joint name="propulsion_fl_joint">

File: src/description/ros2_control/science/science.laser.ros2_control.xacro (robot description, xacro)
@@ -1,5 +1,5 @@
 <?xml version="1.0"?>
 <robot xmlns:xacro="http://www.ros.org/wiki/xacro">
-    <xacro:macro name="laser_ros2_control" params="name can_interface:=can0">
+    <xacro:macro name="laser_ros2_control" params="name can_interface">
         <ros2_control name="${name}" type="system">
             <hardware>

File: src/description/ros2_control/science/science.servo.ros2_control.xacro (robot description, xacro)
@@ -1,5 +1,5 @@
 <?xml version="1.0"?>
 <robot xmlns:xacro="http://www.ros.org/wiki/xacro">
-    <xacro:macro name="servo_ros2_control" params="name">
+    <xacro:macro name="servo_ros2_control" params="name can_interface">
         <ros2_control name="${name}" type="system">
             <hardware>
@@ -8,5 +8,5 @@
                 <param name="logger_rate">5</param> <!-- Hz -->
                 <param name="logger_state">1</param> <!-- 0 for off, 1 for on -->
-                <param name="can_interface">can0</param>
+                <param name="can_interface">${can_interface}</param>
                 <param name="can_id">0x80</param>
             </hardware>

File: src/description/ros2_control/science/science.talon.ros2_control.xacro (robot description, xacro)
@@ -1,5 +1,5 @@
 <?xml version="1.0"?>
 <robot xmlns:xacro="http://www.ros.org/wiki/xacro">
-  <xacro:macro name="talon_ros2_control" params="name">
+  <xacro:macro name="talon_ros2_control" params="name can_interface">
     <ros2_control name="${name}" type="system">
       <hardware>
@@ -8,5 +8,5 @@
         <param name="logger_rate">5</param> <!-- Hz -->
         <param name="logger_state">0</param> <!-- 0 for off, 1 for on -->
-        <param name="can_interface">can0</param>
+        <param name="can_interface">${can_interface}</param>
       </hardware>
       <joint name="talon_auger">

File: src/description/urdf/athena_arm.urdf.xacro (robot description, xacro)
@@ -5,7 +5,7 @@
   <xacro:arg name="use_mock_hardware" default="false"/>
   <xacro:arg name="mock_sensor_commands" default="false"/>
-  <xacro:arg name="sim_gazebo_classic" default="true"/>
-  <xacro:arg name="sim_gazebo" default="true"/>
-  <xacro:arg name="simulation_controllers" default=""/>
+  <xacro:arg name="use_sim" default="false"/>
+  <!-- Derive CAN interface name from use_sim -->
+  <xacro:property name="can_interface" value="${'vcan0' if '$(arg use_sim)' == 'true' else 'can0'}"/>
   <!-- Macro Imports -->
   <!-- Import athena_arm macro -->
@@ -31,5 +31,5 @@
   </xacro:if>
   <xacro:unless value="$(arg use_mock_hardware)"> <!-- HARDWARE -->
-    <xacro:smc_ros2_control name="smc"/>
+    <xacro:smc_ros2_control name="smc" can_interface="${can_interface}"/>
     <ros2_control name="talon_mock" type="system">
       <hardware>
@@ -45,7 +45,7 @@
       </joint>
     </ros2_control>
-    <xacro:rmd_ros2_control name="rmd"/>
-    <xacro:servo_ros2_control name="servo"/>
-    <!-- <xacro:odrive_ros2_control name="odrive"/> -->
+    <xacro:rmd_ros2_control name="rmd" can_interface="${can_interface}"/>
+    <xacro:servo_ros2_control name="servo" can_interface="${can_interface}"/>
+    <!-- <xacro:odrive_ros2_control name="odrive" can_interface="${can_interface}"/> -->
   </xacro:unless>
 </robot>

File: src/description/urdf/athena_drive.urdf.xacro (robot description, xacro)
@@ -5,6 +5,9 @@
   <xacro:arg name="use_mock_hardware" default="false"/>
   <xacro:arg name="mock_sensor_commands" default="false"/>
-  <xacro:arg name="sim_gazebo" default="true"/>
+  <xacro:arg name="sim_gazebo" default="false"/>
   <xacro:arg name="simulation_controllers" default=""/>
+  <xacro:arg name="use_sim" default="false"/>
+  <!-- Derive CAN interface name from use_sim -->
+  <xacro:property name="can_interface" value="${'vcan0' if '$(arg use_sim)' == 'true' else 'can0'}"/>
   <xacro:include filename="$(find description)/urdf/athena_drive/athena_drive_macro.xacro"/>
   <xacro:include filename="$(find description)/urdf/athena_drive/athena_drive_macro.ros2_control.xacro"/>
@@ -52,10 +55,10 @@
   </xacro:if>
   <xacro:unless value="$(arg use_mock_hardware)">
-    <xacro:odrive_ros2_control name="odrive"/>
-    <xacro:rmd_ros2_control name="rmd"/>
+    <xacro:odrive_ros2_control name="odrive" can_interface="${can_interface}"/>
+    <xacro:rmd_ros2_control name="rmd" can_interface="${can_interface}"/>
     <!-- LED status indicator (GPIO-based) -->
     <xacro:led_ros2_control name="status_led" gpio_pin="25"/>
     <!-- Killswitch (CAN-based) -->
-    <xacro:killswitch_ros2_control name="drive_killswitch"/>
+    <xacro:killswitch_ros2_control name="drive_killswitch" can_interface="${can_interface}"/>
   </xacro:unless>
 </robot>

File: src/description/urdf/athena_science.urdf.xacro (robot description, xacro)
@@ -3,4 +3,7 @@
   <xacro:arg name="use_mock_hardware" default="false"/>
   <xacro:arg name="mock_sensor_commands" default="false"/>
+  <xacro:arg name="use_sim" default="false"/>
+  <!-- Derive CAN interface name from use_sim -->
+  <xacro:property name="can_interface" value="${'vcan0' if '$(arg use_sim)' == 'true' else 'can0'}"/>
   <xacro:include filename="$(find description)/ros2_control/science/science.mock.ros2_control.xacro"/>
   <xacro:include filename="$(find description)/ros2_control/science/science.stepper.ros2_control.xacro" />
@@ -20,9 +23,9 @@
     <xacro:stepper_ros2_control name="stepper"/>
     <!-- Import servo ros2_control description -->
-    <xacro:servo_ros2_control name="servo"/>
+    <xacro:servo_ros2_control name="servo" can_interface="${can_interface}"/>
     <!-- Import talon ros2_control description -->
-    <xacro:talon_ros2_control name="talon"/>
+    <xacro:talon_ros2_control name="talon" can_interface="${can_interface}"/>
     <!-- Import laser ros2_control description (CAN-based) -->
-    <xacro:laser_ros2_control name="spectrometry_laser"/>
+    <xacro:laser_ros2_control name="spectrometry_laser" can_interface="${can_interface}"/>
   </xacro:unless>
 </robot>
